File: Mk3 Prototype.sch (EAGLE design)
At the start: 176 parts, among them IC1 BD49XXX, IC2 CC3100, IC3 S25FL216K0PMFI011, IC4 STM32F401V, IC6 AP3419, J1 ZX62-AB-5PA(11), J2 SWD_SHROUD, J7 SFV30R-2STE1HLF, Q1 BSS84W, Q11 BSS84W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

Commit message: moving pins so the lcd has its hardware CS
Parts:
- C69: value 1n -> 0402/1n/10V/X5R; device TiLDA Mk3 Parts:C-EUC1206K -> TiLDA Mk3 Parts:C-EUC0402-SMALLER
Connections:
- net TIM4_CH4 renamed TIM11_CH1
- removed net LCD_!CS: IC4_PB.PB4, J7.CS1B
- removed net TIM2_CH1: IC4_PA.PA15, U4.D6
- removed net TIM2_CH3: IC4_PB.PB10, U4.D5
- new net N$50: SV1.2
- new net SPI3_NSS: IC4_PA.PA15, J7.CS1B
- new net TIM10_CH1: IC4_PB.PB8, JP4.2, U4.D9
- new net TIM4_CH2: IC4_PD.PD13, U4.D5
- net JOY_RIGHT: now also IC4_PD.PD8; no longer IC4_PD.PD13
- net MOM_DWN: now also IC4_PE.PE10; no longer IC4_PE.PE8
- net TIM4_CH3: now also IC4_PD.PD14, U4.D6; no longer IC4_PB.PB8, JP4.2, U4.D9
Other:
- note added: "tim2_ch1"
Changed lines of the file:
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@@
 <part name="IC1" library="TiLDA Mk3 Parts" deviceset="BD49XXX" device=""/>
 <part name="GND98" library="TiLDA Mk3 Parts" deviceset="GND" device=""/>
-<part name="C69" library="TiLDA Mk3 Parts" deviceset="C-EU" device="C1206K" value="1n"/>
 <part name="GND99" library="TiLDA Mk3 Parts" deviceset="GND" device=""/>
+<part name="C69" library="TiLDA Mk3 Parts" deviceset="C-EU" device="C0402-SMALLER" value="0402/1n/10V/X5R"/>
 </parts>
 <sheets>
@@
 <wire x1="581.66" y1="10.16" x2="581.66" y2="33.02" width="0.1524" layer="97"/>
 <text x="297.18" y="243.84" size="1.778" layer="91">- needed with low voltage cutoff?</text>
+<text x="-20.32" y="177.8" size="1.778" layer="91">tim2_ch1</text>
 </plain>
 <instances>
@@
 <instance part="IC1" gate="G$1" x="576.58" y="35.56"/>
 <instance part="GND98" gate="1" x="566.42" y="27.94"/>
-<instance part="C69" gate="G$1" x="591.82" y="27.94"/>
 <instance part="GND99" gate="1" x="591.82" y="20.32"/>
+<instance part="C69" gate="G$1" x="591.82" y="27.94"/>
 </instances>
 <busses>
@@
 </segment>
 <segment>
-<pinref part="C69" gate="G$1" pin="2"/>
 <pinref part="GND99" gate="1" pin="GND"/>
+<pinref part="C69" gate="G$1" pin="2"/>
 </segment>
 </net>
@@
 </segment>
 </net>
-<net name="LCD_!CS" class="0">
-<segment>
-<pinref part="J7" gate="G$1" pin="CS1B"/>
-<wire x1="360.68" y1="246.38" x2="363.22" y2="246.38" width="0.1524" layer="91"/>
-<label x="360.68" y="246.38" size="1.778" layer="95" rot="MR0"/>
-</segment>
-<segment>
-<pinref part="IC4" gate="_PB" pin="PB4"/>
-<wire x1="68.58" y1="193.04" x2="71.12" y2="193.04" width="0.1524" layer="91"/>
-<label x="71.12" y="193.04" size="1.778" layer="95"/>
-</segment>
-</net>
 <net name="LCD_POWER" class="0">
 <segment>
@@
 </segment>
 </net>
-<net name="TIM4_CH4" class="0">
-<segment>
-<wire x1="68.58" y1="177.8" x2="71.12" y2="177.8" width="0.1524" layer="91"/>
-<label x="71.12" y="177.8" size="1.778" layer="95"/>
-<pinref part="IC4" gate="_PB" pin="PB9"/>
-</segment>
-<segment>
-<wire x1="304.8" y1="50.8" x2="307.34" y2="50.8" width="0.1524" layer="91"/>
-<label x="304.8" y="50.8" size="1.778" layer="95" rot="MR0"/>
-<pinref part="U4" gate="G$1" pin="D10"/>
-<pinref part="JP4" gate="G$1" pin="3"/>
-<junction x="307.34" y="50.8"/>
-</segment>
-</net>
 <net name="I2C_SCL" class="0">
 <segment>
@@
 </segment>
 </net>
-<net name="TIM2_CH1" class="0">
-<segment>
-<wire x1="33.02" y1="162.56" x2="30.48" y2="162.56" width="0.1524" layer="91"/>
-<pinref part="IC4" gate="_PA" pin="PA15"/>
-<label x="33.02" y="162.56" size="1.778" layer="95"/>
-</segment>
-<segment>
-<wire x1="304.8" y1="63.5" x2="307.34" y2="63.5" width="0.1524" layer="91"/>
-<label x="304.8" y="63.5" size="1.778" layer="95" rot="MR0"/>
-<pinref part="U4" gate="G$1" pin="D6"/>
-</segment>
-</net>
-<net name="TIM4_CH3" class="0">
+<net name="TIM10_CH1" class="0">
 <segment>
 <wire x1="71.12" y1="180.34" x2="68.58" y2="180.34" width="0.1524" layer="91"/>
@@
 </segment>
 </net>
-<net name="TIM2_CH3" class="0">
-<segment>
-<wire x1="71.12" y1="175.26" x2="68.58" y2="175.26" width="0.1524" layer="91"/>
-<label x="71.12" y="175.26" size="1.778" layer="95"/>
-<pinref part="IC4" gate="_PB" pin="PB10"/>
-</segment>
-<segment>
-<wire x1="304.8" y1="66.04" x2="307.34" y2="66.04" width="0.1524" layer="91"/>
-<label x="304.8" y="66.04" size="1.778" layer="95" rot="MR0"/>
-<pinref part="U4" gate="G$1" pin="D5"/>
-</segment>
-</net>
 <net name="USART6_TX" class="0">
 <segment>
@@
 </segment>
 <segment>
-<pinref part="IC4" gate="_PD" pin="PD13"/>
-<wire x1="93.98" y1="104.14" x2="104.14" y2="104.14" width="0.1524" layer="91"/>
-<label x="96.52" y="104.14" size="1.778" layer="95"/>
+<pinref part="IC4" gate="_PD" pin="PD8"/>
+<wire x1="93.98" y1="116.84" x2="104.14" y2="116.84" width="0.1524" layer="91"/>
+<label x="96.52" y="116.84" size="1.778" layer="95"/>
 </segment>
 </net>
@@
 </segment>
 <segment>
-<pinref part="IC4" gate="_PE" pin="PE8"/>
-<wire x1="93.98" y1="53.34" x2="101.6" y2="53.34" width="0.1524" layer="91"/>
-<label x="99.06" y="53.34" size="1.778" layer="95"/>
+<pinref part="IC4" gate="_PE" pin="PE10"/>
+<wire x1="93.98" y1="48.26" x2="99.06" y2="48.26" width="0.1524" layer="91"/>
+<label x="99.06" y="48.26" size="1.778" layer="95"/>
 </segment>
 </net>
@@
 <wire x1="594.36" y1="40.64" x2="594.36" y2="35.56" width="0.1524" layer="91"/>
 <pinref part="IC1" gate="G$1" pin="OUT"/>
-<pinref part="C69" gate="G$1" pin="1"/>
 <wire x1="591.82" y1="30.48" x2="591.82" y2="35.56" width="0.1524" layer="91"/>
 <wire x1="591.82" y1="35.56" x2="594.36" y2="35.56" width="0.1524" layer="91"/>
 <junction x="591.82" y="35.56"/>
+<pinref part="C69" gate="G$1" pin="1"/>
+</segment>
+</net>
+<net name="SPI3_NSS" class="0">
+<segment>
+<wire x1="33.02" y1="162.56" x2="30.48" y2="162.56" width="0.1524" layer="91"/>
+<pinref part="IC4" gate="_PA" pin="PA15"/>
+<label x="33.02" y="162.56" size="1.778" layer="95"/>
+</segment>
+<segment>
+<pinref part="J7" gate="G$1" pin="CS1B"/>
+<wire x1="360.68" y1="246.38" x2="363.22" y2="246.38" width="0.1524" layer="91"/>
+<label x="360.68" y="246.38" size="1.778" layer="95" rot="MR0"/>
+</segment>
+</net>
+<net name="TIM11_CH1" class="0">
+<segment>
+<wire x1="68.58" y1="177.8" x2="71.12" y2="177.8" width="0.1524" layer="91"/>
+<label x="71.12" y="177.8" size="1.778" layer="95"/>
+<pinref part="IC4" gate="_PB" pin="PB9"/>
+</segment>
+<segment>
+<wire x1="304.8" y1="50.8" x2="307.34" y2="50.8" width="0.1524" layer="91"/>
+<label x="304.8" y="50.8" size="1.778" layer="95" rot="MR0"/>
+<pinref part="U4" gate="G$1" pin="D10"/>
+<pinref part="JP4" gate="G$1" pin="3"/>
+<junction x="307.34" y="50.8"/>
+</segment>
+</net>
+<net name="TIM4_CH2" class="0">
+<segment>
+<pinref part="IC4" gate="_PD" pin="PD13"/>
+<wire x1="93.98" y1="104.14" x2="104.14" y2="104.14" width="0.1524" layer="91"/>
+<label x="96.52" y="104.14" size="1.778" layer="95"/>
+</segment>
+<segment>
+<wire x1="304.8" y1="66.04" x2="307.34" y2="66.04" width="0.1524" layer="91"/>
+<label x="304.8" y="66.04" size="1.778" layer="95" rot="MR0"/>
+<pinref part="U4" gate="G$1" pin="D5"/>
+</segment>
+</net>
+<net name="TIM4_CH3" class="0">
+<segment>
+<pinref part="IC4" gate="_PD" pin="PD14"/>
+<wire x1="93.98" y1="101.6" x2="104.14" y2="101.6" width="0.1524" layer="91"/>
+<label x="96.52" y="101.6" size="1.778" layer="95"/>
+</segment>
+<segment>
+<wire x1="304.8" y1="63.5" x2="307.34" y2="63.5" width="0.1524" layer="91"/>
+<label x="304.8" y="63.5" size="1.778" layer="95" rot="MR0"/>
+<pinref part="U4" gate="G$1" pin="D6"/>
+</segment>
+</net>
+<net name="N$50" class="0">
+<segment>
+<pinref part="SV1" gate="G$1" pin="2"/>
+<wire x1="528.32" y1="101.6" x2="530.86" y2="101.6" width="0.1524" layer="91"/>
+<wire x1="530.86" y1="101.6" x2="530.86" y2="109.22" width="0.1524" layer="91"/>
+<wire x1="530.86" y1="109.22" x2="523.24" y2="109.22" width="0.1524" layer="91"/>
+<wire x1="523.24" y1="109.22" x2="523.24" y2="129.54" width="0.1524" layer="91"/>
 </segment>
 </net>
