File: Mk3 Prototype.sch (EAGLE design)
At the start: 188 parts, among them IC1 BD49XXX, IC2 NCP1529MU, IC3 STM32F401V, IC4 CC3100, IC5 S25FL216K0PMFI011, J1 ZX62-AB-5PA(11), J2 SFV30R-2STE1HLF, J3 SWD_SHROUD, Q1 DMMT5401, Q2 NTR4101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

Commit message: added comment about switch
Other:
- note added: "sort out power switch"
Changed lines of the file:
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@@
 <text x="129.286" y="199.136" size="1.778" layer="91" rot="R90">low ESR</text>
 <text x="797.56" y="170.18" size="2.54" layer="94">move esp decoupling cap to vcc pin</text>
+<text x="797.56" y="162.56" size="2.54" layer="94">sort out power switch</text>
 </plain>
 <instances>

Commit message: changing 4x0603->2x0805, power mosfet, lcd mosfet
Parts:
- removed C38, C45, C48, C61: 0603/10u/6.3V/X5R, TiLDA Mk3 Parts:C-EUC0603K-SMALL
- added C27, C40: 0805/22u/??V/X5R, passives-7351:CAPACITOR0805-N
- added Q6: NTR4101, TiLDA Mk3 Parts:MOSFET-P-SOT23
- added R44: 0402/1R/5%, TiLDA Mk3 Parts:R-EU_R0402-SMALLER
- added R45: 0402/220k/5%, TiLDA Mk3 Parts:R-EU_R0402-SMALLER
- Q4: value BSS84W -> NTR4101; device TiLDA Mk3 Parts:MOSFET-P-SC70-3 -> TiLDA Mk3 Parts:MOSFET-P-SOT23
Connections:
- new net LCD_VCC: J2.C86, J2.D0, J2.D1, J2.D2, J2.D3, J2.D4, J2.D5, J2.RD, J2.VDD, J2.WR, Q4.D
- new net N$53: Q4.S, R44.2
- new net N$54: Q6.G, R45.2, S5.S
- net +3V3: now also R44.1; no longer J2.C86, J2.D0, J2.D1, J2.D2, J2.D3, J2.D4, J2.D5, J2.RD, J2.VDD, J2.WR
- net GND: now also C27.1, C40.1, S5.P; no longer C38.1, C45.1, C48.1, C61.1
- net LCD_POWER: now also IC3_PB.PB4
- net N$15: now also Q6.S, R45.1; no longer S5.S
- net N$17: now also C27.2, C40.2; no longer C38.2, C45.2, C48.2, C61.2
- net V_UNREG: now also Q6.D; no longer S5.P
Other:
- note added: "NOTE: need to disable spi when screen power is off"
- moved on the sheet: S5

Commit message: wiring cc programming interface to stm32
Parts:
- added R46: 0402/10K/5%, TiLDA Mk3 Parts:R-EU_R0402-SMALLER
- added TP12, TP13: TPB1,27, TiLDA Mk3 Parts:TPB1,27
Connections:
- removed net N$46: IC4_UART.TX, SV1.3
- removed net N$47: IC4_UART.RX, SV1.2
- new net N$40: IC4_UART.TX, R46.2, SV1.3
- net +3V3: now also TP12.TP
- net N$53: now also TP13.TP
- net USART6_RX: now also R46.1
- net USART6_TX: now also IC4_UART.RX, SV1.2
- net WIFI_!RESET: now also IC3_PE.PE8
Changed lines of the file:
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@@
 <part name="C27" library="passives-7351" deviceset="CAPACITOR" device="0805-N" value="0805/22u/??V/X5R"/>
 <part name="C40" library="passives-7351" deviceset="CAPACITOR" device="0805-N" value="0805/22u/??V/X5R"/>
+<part name="TP12" library="TiLDA Mk3 Parts" deviceset="TP" device="B1,27"/>
+<part name="TP13" library="TiLDA Mk3 Parts" deviceset="TP" device="B1,27"/>
+<part name="R46" library="TiLDA Mk3 Parts" deviceset="R-EU_" device="R0402-SMALLER" value="0402/10K/5%"/>
 </parts>
 <sheets>
@@
 <attribute name="VALUE" x="442.341" y="220.98" size="1.778" layer="96" rot="R270"/>
 </instance>
+<instance part="TP12" gate="G$1" x="314.96" y="231.14" smashed="yes">
+<attribute name="NAME" x="313.69" y="232.41" size="1.778" layer="95"/>
+</instance>
+<instance part="TP13" gate="G$1" x="325.12" y="231.14" smashed="yes">
+<attribute name="NAME" x="323.85" y="232.41" size="1.778" layer="95"/>
+</instance>
+<instance part="R46" gate="G$1" x="622.3" y="190.5" smashed="yes" rot="R90">
+<attribute name="NAME" x="620.8014" y="186.69" size="1.778" layer="95" rot="R90"/>
+<attribute name="VALUE" x="617.982" y="179.07" size="1.778" layer="96" rot="R90"/>
+</instance>
 </instances>
 <busses>
@@
 <pinref part="S6" gate="G$1" pin="1"/>
 </segment>
+<segment>
+<pinref part="IC3" gate="_PE" pin="PE8"/>
+<wire x1="93.98" y1="53.34" x2="99.06" y2="53.34" width="0.1524" layer="91"/>
+<label x="96.52" y="53.34" size="1.778" layer="95"/>
+</segment>
 </net>
 <net name="WIFI_FORCE_AP" class="0">
@@
 <pinref part="R44" gate="G$1" pin="1"/>
 <pinref part="+3V9" gate="G$1" pin="+3V3"/>
-<wire x1="314.96" y1="226.06" x2="312.42" y2="226.06" width="0.1524" layer="91"/>
+<pinref part="TP12" gate="G$1" pin="TP"/>
+<wire x1="314.96" y1="228.6" x2="314.96" y2="226.06" width="0.1524" layer="91"/>
+<wire x1="312.42" y1="226.06" x2="314.96" y2="226.06" width="0.1524" layer="91"/>
+<junction x="314.96" y="226.06"/>
 </segment>
 </net>
@@
 </segment>
 </net>
-<net name="N$40" class="0">
-<segment>
-<wire x1="314.96" y1="236.22" x2="320.04" y2="236.22" width="0.1524" layer="91"/>
-<wire x1="320.04" y1="236.22" x2="325.12" y2="231.14" width="0.1524" layer="91"/>
-</segment>
-</net>
 <net name="MCO1" class="0">
 <segment>
@@
 </segment>
 </net>
-<net name="N$46" class="0">
-<segment>
-<pinref part="IC4" gate="_UART" pin="TX"/>
-<wire x1="637.54" y1="236.22" x2="624.84" y2="236.22" width="0.1524" layer="91"/>
-<pinref part="SV1" gate="G$1" pin="3"/>
-</segment>
-</net>
-<net name="N$47" class="0">
-<segment>
-<pinref part="IC4" gate="_UART" pin="RX"/>
-<wire x1="624.84" y1="233.68" x2="637.54" y2="233.68" width="0.1524" layer="91"/>
-<pinref part="SV1" gate="G$1" pin="2"/>
-</segment>
-</net>
 <net name="USB_ID_" class="0">
 <segment>
@@
 <segment>
 <pinref part="X1" gate="G$1" pin="URXD"/>
-<wire x1="655.32" y1="162.56" x2="642.62" y2="162.56" width="0.1524" layer="91"/>
-<label x="642.62" y="162.56" size="1.778" layer="95"/>
+<label x="599.44" y="162.56" size="1.778" layer="95"/>
+<wire x1="655.32" y1="162.56" x2="624.84" y2="162.56" width="0.1524" layer="91"/>
+<wire x1="624.84" y1="162.56" x2="599.44" y2="162.56" width="0.1524" layer="91"/>
+<wire x1="624.84" y1="162.56" x2="624.84" y2="213.36" width="0.1524" layer="91"/>
+<wire x1="624.84" y1="213.36" x2="632.46" y2="213.36" width="0.1524" layer="91"/>
+<pinref part="IC4" gate="_UART" pin="RX"/>
+<wire x1="624.84" y1="233.68" x2="632.46" y2="233.68" width="0.1524" layer="91"/>
+<pinref part="SV1" gate="G$1" pin="2"/>
+<wire x1="632.46" y1="233.68" x2="637.54" y2="233.68" width="0.1524" layer="91"/>
+<wire x1="632.46" y1="213.36" x2="632.46" y2="233.68" width="0.1524" layer="91"/>
+<junction x="632.46" y="233.68"/>
+<junction x="624.84" y="162.56"/>
 </segment>
 </net>
@@
 <segment>
 <pinref part="X1" gate="G$1" pin="UTXD"/>
-<wire x1="642.62" y1="160.02" x2="655.32" y2="160.02" width="0.1524" layer="91"/>
-<label x="642.62" y="160.02" size="1.778" layer="95"/>
+<label x="599.44" y="160.02" size="1.778" layer="95"/>
+<wire x1="655.32" y1="160.02" x2="622.3" y2="160.02" width="0.1524" layer="91"/>
+<pinref part="R46" gate="G$1" pin="1"/>
+<wire x1="622.3" y1="160.02" x2="599.44" y2="160.02" width="0.1524" layer="91"/>
+<wire x1="622.3" y1="185.42" x2="622.3" y2="160.02" width="0.1524" layer="91"/>
+<junction x="622.3" y="160.02"/>
 </segment>
 </net>
@@
 <segment>
 <pinref part="R44" gate="G$1" pin="2"/>
-<wire x1="325.12" y1="226.06" x2="327.66" y2="226.06" width="0.1524" layer="91"/>
 <pinref part="Q4" gate="G$1" pin="S"/>
+<pinref part="TP13" gate="G$1" pin="TP"/>
+<wire x1="325.12" y1="228.6" x2="325.12" y2="226.06" width="0.1524" layer="91"/>
+<wire x1="325.12" y1="226.06" x2="327.66" y2="226.06" width="0.1524" layer="91"/>
+<junction x="325.12" y="226.06"/>
 </segment>
 </net>
@@
 </segment>
 </net>
+<net name="N$40" class="0">
+<segment>
+<pinref part="IC4" gate="_UART" pin="TX"/>
+<pinref part="SV1" gate="G$1" pin="3"/>
+<wire x1="637.54" y1="236.22" x2="629.92" y2="236.22" width="0.1524" layer="91"/>
+<wire x1="629.92" y1="236.22" x2="624.84" y2="236.22" width="0.1524" layer="91"/>
+<junction x="629.92" y="236.22"/>
+<wire x1="629.92" y1="215.9" x2="629.92" y2="236.22" width="0.1524" layer="91"/>
+<wire x1="622.3" y1="215.9" x2="629.92" y2="215.9" width="0.1524" layer="91"/>
+<pinref part="R46" gate="G$1" pin="2"/>
+<wire x1="622.3" y1="195.58" x2="622.3" y2="215.9" width="0.1524" layer="91"/>
+</segment>
+</net>

Commit message: lots of cleaing up, silk screen, drc fixes
Parts:
- removed JP2: (no value), TiLDA Mk3 Parts:PINHEAD_PINHD-2X5PASSO127
- removed Y1: AH316M245001-T, TiLDA Mk3 Parts:AH316M245001-T
- D2, D3: device TiLDA Mk3 Parts:DIODE-SOD123 -> TiLDA Mk3 Parts:DIODESOD-323F
- renumbered JP1 to SW1, R13 to Z2, R17 to Z3, R20 to Z1
Other:
- note added: "RETHINK"
Changed lines of the file:
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@@
 <?xml version="1.0" encoding="utf-8"?>
 <!DOCTYPE eagle SYSTEM "eagle.dtd">
-<eagle version="6.5.0">
+<eagle version="6.6.0">
 <drawing>
 <settings>
@@
 <part name="GND9" library="TiLDA Mk3 Parts" deviceset="GND" device=""/>
 <part name="GND10" library="TiLDA Mk3 Parts" deviceset="GND" device=""/>
-<part name="Y1" library="TiLDA Mk3 Parts" deviceset="AH316M245001-T" device=""/>
-<part name="GND11" library="TiLDA Mk3 Parts" deviceset="GND" device=""/>
 <part name="R31" library="TiLDA Mk3 Parts" deviceset="R-EU_" device="R0402-SMALLER" value="0402/100K/5%"/>
 <part name="R39" library="TiLDA Mk3 Parts" deviceset="R-EU_" device="R0402-SMALLER" value="0402/100K/5%"/>
@@
 <part name="+3V3" library="supply1" deviceset="+3V3" device=""/>
 <part name="+3V4" library="supply1" deviceset="+3V3" device=""/>
-<part name="JP1" library="TiLDA Mk3 Parts" deviceset="JOYSTICK_MINI" device="_MULTICOMP"/>
+<part name="SW1" library="TiLDA Mk3 Parts" deviceset="JOYSTICK_MINI" device="_MULTICOMP"/>
 <part name="S2" library="Mine" deviceset="SWITCH-MOMENTARY-2" device=""/>
 <part name="S1" library="Mine" deviceset="SWITCH-MOMENTARY-2" device=""/>
@@
 <part name="GND79" library="TiLDA Mk3 Parts" deviceset="GND" device=""/>
 <part name="L3" library="TiLDA Mk3 Parts" deviceset="WE-CBF" device="_0805" value="Bead"/>
-<part name="JP2" library="TiLDA Mk3 Parts" deviceset="PINHEAD_PINHD-2X5" device="PASSO127"/>
 <part name="G1" library="dtb" deviceset="GND-LOOP" device="" value="GND-LOOP"/>
 <part name="GND56" library="TiLDA Mk3 Parts" deviceset="GND" device=""/>
@@
 <part name="C6" library="passives-7351" deviceset="CAPACITOR" device="0805-N" value="0805/10u/10V/X5R"/>
 <part name="GND94" library="TiLDA Mk3 Parts" deviceset="GND" device=""/>
-<part name="D3" library="TiLDA Mk3 Parts" deviceset="DIODE-" device="SOD123"/>
-<part name="D2" library="TiLDA Mk3 Parts" deviceset="DIODE-" device="SOD123"/>
+<part name="D3" library="TiLDA Mk3 Parts" deviceset="DIODE" device="SOD-323F"/>
+<part name="D2" library="TiLDA Mk3 Parts" deviceset="DIODE" device="SOD-323F"/>
 <part name="SJ1" library="SparkFun-Passives" deviceset="JUMPER-PAD-2-NO" device="YES_SILK"/>
 <part name="JP4" library="SparkFun-Connectors" deviceset="M10" device="SILK_FEMALE_PTH"/>
@@
 <part name="GND105" library="TiLDA Mk3 Parts" deviceset="GND" device=""/>
 <part name="+3V24" library="supply1" deviceset="+3V3" device=""/>
-<part name="R20" library="TiLDA Mk3 Parts" deviceset="VARISTOR" device="CN0603"/>
-<part name="R13" library="TiLDA Mk3 Parts" deviceset="VARISTOR" device="CN0603"/>
-<part name="R17" library="TiLDA Mk3 Parts" deviceset="VARISTOR" device="CN0603"/>
+<part name="Z1" library="TiLDA Mk3 Parts" deviceset="VARISTOR" device="CN0603"/>
+<part name="Z2" library="TiLDA Mk3 Parts" deviceset="VARISTOR" device="CN0603"/>
+<part name="Z3" library="TiLDA Mk3 Parts" deviceset="VARISTOR" device="CN0603"/>
 <part name="GND106" library="TiLDA Mk3 Parts" deviceset="GND" device=""/>
 <part name="+3V25" library="supply1" deviceset="+3V3" device=""/>
@@
 <text x="320.04" y="251.46" size="1.778" layer="97">NOTE: need to disable spi
 when screen power is off</text>
+<text x="378.46" y="60.96" size="1.778" layer="91" rot="R90">RETHINK</text>
 </plain>
 <instances>
@@
 <instance part="GND9" gate="1" x="716.28" y="213.36"/>
 <instance part="GND10" gate="1" x="736.6" y="213.36"/>
-<instance part="Y1" gate="G$1" x="754.38" y="246.38" smashed="yes" rot="MR270">
-<attribute name="VALUE" x="759.46" y="246.38" size="1.778" layer="96"/>
-<attribute name="NAME" x="759.46" y="249.682" size="1.778" layer="95"/>
-</instance>
-<instance part="GND11" gate="1" x="759.46" y="241.3" rot="R90"/>
 <instance part="R31" gate="G$1" x="762" y="129.54" rot="R270"/>
 <instance part="R39" gate="G$1" x="772.16" y="129.54" rot="R270"/>
@@
 <instance part="+3V3" gate="G$1" x="375.92" y="48.26" rot="R270"/>
 <instance part="+3V4" gate="G$1" x="10.16" y="27.94"/>
-<instance part="JP1" gate="G$1" x="330.2" y="129.54"/>
+<instance part="SW1" gate="G$1" x="330.2" y="129.54"/>
 <instance part="S2" gate="G$1" x="337.82" y="104.14" smashed="yes">
 <attribute name="NAME" x="335.28" y="106.68" size="1.778" layer="95"/>
@@
 <instance part="GND79" gate="1" x="254" y="177.8"/>
 <instance part="L3" gate="G$1" x="139.7" y="195.58"/>
-<instance part="JP2" gate="G$1" x="60.96" y="17.78"/>
 <instance part="G1" gate="G$1" x="673.1" y="17.78"/>
 <instance part="GND56" gate="1" x="670.56" y="10.16"/>
@@
 <instance part="GND105" gate="1" x="152.4" y="86.36" rot="R90"/>
 <instance part="+3V24" gate="G$1" x="119.38" y="86.36" rot="R90"/>
-<instance part="R20" gate="G$1" x="205.74" y="93.98" rot="R90"/>
-<instance part="R13" gate="G$1" x="210.82" y="93.98" rot="R90"/>
-<instance part="R17" gate="G$1" x="215.9" y="93.98" rot="R90"/>
+<instance part="Z1" gate="G$1" x="205.74" y="93.98" rot="R90"/>
+<instance part="Z2" gate="G$1" x="210.82" y="93.98" rot="R90"/>
+<instance part="Z3" gate="G$1" x="215.9" y="93.98" rot="R90"/>
 <instance part="GND106" gate="1" x="210.82" y="83.82"/>
 <instance part="+3V25" gate="G$1" x="457.2" y="132.08"/>
@@
 </segment>
 <segment>
-<pinref part="R17" gate="G$1" pin="2"/>
+<pinref part="Z3" gate="G$1" pin="2"/>
 <wire x1="215.9" y1="88.9" x2="215.9" y2="86.36" width="0.1524" layer="91"/>
 <wire x1="215.9" y1="86.36" x2="210.82" y2="86.36" width="0.1524" layer="91"/>
-<pinref part="R13" gate="G$1" pin="2"/>
+<pinref part="Z2" gate="G$1" pin="2"/>
 <wire x1="210.82" y1="86.36" x2="210.82" y2="88.9" width="0.1524" layer="91"/>
 <wire x1="210.82" y1="86.36" x2="205.74" y2="86.36" width="0.1524" layer="91"/>
-<pinref part="R20" gate="G$1" pin="2"/>
+<pinref part="Z1" gate="G$1" pin="2"/>
 <wire x1="205.74" y1="86.36" x2="205.74" y2="88.9" width="0.1524" layer="91"/>
 <junction x="210.82" y="86.36"/>
@@
 </segment>
 </net>
-<net name="N$3" class="1">
+<net name="N$3" class="0">
 <segment>
 <pinref part="FL1" gate="G$1" pin="IN"/>
@@
 </segment>
 <segment>
-<pinref part="JP1" gate="G$1" pin="COM"/>
+<pinref part="SW1" gate="G$1" pin="COM"/>
 <pinref part="+3V14" gate="G$1" pin="+3V3"/>
 </segment>
@@
 <wire x1="205.74" y1="114.3" x2="205.74" y2="101.6" width="0.1524" layer="91"/>
 <wire x1="205.74" y1="101.6" x2="228.6" y2="101.6" width="0.1524" layer="91"/>
-<pinref part="R20" gate="G$1" pin="1"/>
+<pinref part="Z1" gate="G$1" pin="1"/>
 <wire x1="205.74" y1="99.06" x2="205.74" y2="101.6" width="0.1524" layer="91"/>
 <junction x="205.74" y="101.6"/>
@@
 </segment>
 <segment>
-<pinref part="JP1" gate="G$1" pin="CENT"/>
+<pinref part="SW1" gate="G$1" pin="CENT"/>
 <wire x1="342.9" y1="127" x2="353.06" y2="127" width="0.1524" layer="91"/>
 <label x="347.98" y="127" size="1.778" layer="95"/>
@@
 <pinref part="J1" gate="G$1" pin="D-"/>
 <wire x1="213.36" y1="119.38" x2="208.28" y2="119.38" width="0.1524" layer="91"/>
-<pinref part="R13" gate="G$1" pin="1"/>
+<pinref part="Z2" gate="G$1" pin="1"/>
 <wire x1="208.28" y1="119.38" x2="193.04" y2="119.38" width="0.1524" layer="91"/>
 <wire x1="210.82" y1="99.06" x2="210.82" y2="106.68" width="0.1524" layer="91"/>
@@
 <wire x1="210.82" y1="116.84" x2="210.82" y2="109.22" width="0.1524" layer="91"/>
 <wire x1="210.82" y1="109.22" x2="215.9" y2="109.22" width="0.1524" layer="91"/>
-<pinref part="R17" gate="G$1" pin="1"/>
+<pinref part="Z3" gate="G$1" pin="1"/>
 <wire x1="215.9" y1="109.22" x2="215.9" y2="99.06" width="0.1524" layer="91"/>
 <junction x="210.82" y="116.84"/>
 </segment>
 </net>
-<net name="D_N" class="2">
+<net name="D_N" class="0">
 <segment>
 <pinref part="R23" gate="G$1" pin="1"/>
@@
 </segment>
 </net>
-<net name="D_P" class="2">
+<net name="D_P" class="0">
 <segment>
 <pinref part="R25" gate="G$1" pin="1"/>
@@
 <net name="JOY_UP" class="0">
 <segment>
-<pinref part="JP1" gate="G$1" pin="UP"/>
+<pinref part="SW1" gate="G$1" pin="UP"/>
 <wire x1="317.5" y1="132.08" x2="309.88" y2="132.08" width="0.1524" layer="91"/>
 <label x="312.42" y="132.08" size="1.778" layer="95" rot="MR0"/>
@@
 <net name="JOY_DWN" class="0">
 <segment>
-<pinref part="JP1" gate="G$1" pin="DOWN"/>
+<pinref part="SW1" gate="G$1" pin="DOWN"/>
 <wire x1="317.5" y1="129.54" x2="309.88" y2="129.54" width="0.1524" layer="91"/>
 <label x="312.42" y="129.54" size="1.778" layer="95" rot="MR0"/>
@@
 <net name="JOY_LEFT" class="0">
 <segment>
-<pinref part="JP1" gate="G$1" pin="LEFT"/>
+<pinref part="SW1" gate="G$1" pin="LEFT"/>
 <wire x1="342.9" y1="132.08" x2="353.06" y2="132.08" width="0.1524" layer="91"/>
 <label x="347.98" y="132.08" size="1.778" layer="95"/>
@@
 <net name="JOY_RIGHT" class="0">
 <segment>
-<pinref part="JP1" gate="G$1" pin="RIGHT"/>
+<pinref part="SW1" gate="G$1" pin="RIGHT"/>
 <wire x1="342.9" y1="129.54" x2="353.06" y2="129.54" width="0.1524" layer="91"/>
 <label x="347.98" y="129.54" size="1.778" layer="95"/>
@@
 </segment>
 </net>
+<net name="N$46" class="0">
+<segment>
+<wire x1="795.02" y1="165.1" x2="845.82" y2="162.56" width="0.1524" layer="91"/>
+</segment>
+</net>
+<net name="N$47" class="0">
+<segment>
+<wire x1="845.82" y1="167.64" x2="795.02" y2="162.56" width="0.1524" layer="91"/>
+</segment>
+</net>
+<net name="N$55" class="0">
+<segment>
+<wire x1="797.56" y1="172.72" x2="873.76" y2="170.18" width="0.1524" layer="91"/>
+</segment>
+</net>
+<net name="N$62" class="0">
+<segment>
+<wire x1="873.76" y1="175.26" x2="797.56" y2="170.18" width="0.1524" layer="91"/>
+</segment>
+</net>

Commit message: more little bits and pieces; current shunt on esp
Parts:
- added R13: 0402/0.1R/5%, TiLDA Mk3 Parts:R-EU_R0402-SMALLER
- added TP11, TP14: TPB1,27, TiLDA Mk3 Parts:TPB1,27
Connections:
- new net VCC: C41.2, R13.2, TP14.TP, X1.VCC
- net +3V3: now also R13.1, TP11.TP; no longer C41.2, X1.VCC
Other:
- note removed: "add testpoints"
- note removed: "connect these three"
- moved on the sheet: L2, L3
Changed lines of the file:
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@@
 <part name="TP13" library="TiLDA Mk3 Parts" deviceset="TP" device="B1,27"/>
 <part name="R46" library="TiLDA Mk3 Parts" deviceset="R-EU_" device="R0402-SMALLER" value="0402/10K/5%"/>
+<part name="R13" library="TiLDA Mk3 Parts" deviceset="R-EU_" device="R0402-SMALLER" value="0402/0.1R/5%"/>
+<part name="TP11" library="TiLDA Mk3 Parts" deviceset="TP" device="B1,27"/>
+<part name="TP14" library="TiLDA Mk3 Parts" deviceset="TP" device="B1,27"/>
 </parts>
 <sheets>
@@
 to a ftdi header for debug</text>
 <text x="797.56" y="223.52" size="2.54" layer="94">SDIO_SW can be easily changed away from pin PC13</text>
-<text x="628.904" y="126.238" size="1.778" layer="91" rot="R90">connect these three </text>
 <text x="797.56" y="215.9" size="2.54" layer="94">check DMA channel conflicts</text>
 <text x="797.56" y="208.28" size="2.54" layer="94">check ESP pin connections</text>
@@
 `improve heat dissipation and yield'</text>
 <wire x1="518.16" y1="271.78" x2="518.16" y2="243.84" width="0.1524" layer="97"/>
-<text x="640.08" y="157.48" size="1.778" layer="91" rot="R90">add testpoints</text>
 <text x="612.14" y="264.16" size="1.778" layer="91">http://processors.wiki.ti.com/index.php/CC3100_Production_Line_Guide#Programming_the_CC3100_QFN_in_the_Production_Line</text>
 <text x="797.56" y="193.04" size="2.54" layer="94">aref arrangment, consider to allow Aref changing on gpio</text>
@@
 </instance>
 <instance part="GND80" gate="1" x="673.1" y="106.68"/>
-<instance part="+3V11" gate="G$1" x="673.1" y="172.72"/>
+<instance part="+3V11" gate="G$1" x="655.32" y="170.18" rot="R90"/>
 <instance part="+3V12" gate="G$1" x="637.54" y="144.78" smashed="yes" rot="R90">
 <attribute name="VALUE" x="636.778" y="145.796" size="1.778" layer="96" rot="R180"/>
@@
 <attribute name="VALUE" x="617.982" y="179.07" size="1.778" layer="96" rot="R90"/>
 </instance>
+<instance part="R13" gate="G$1" x="665.48" y="170.18"/>
+<instance part="TP11" gate="G$1" x="660.4" y="172.72" smashed="yes">
+<attribute name="NAME" x="659.13" y="173.99" size="1.778" layer="95"/>
+</instance>
+<instance part="TP14" gate="G$1" x="673.1" y="172.72" smashed="yes">
+<attribute name="NAME" x="671.83" y="173.99" size="1.778" layer="95"/>
+</instance>
 </instances>
 <busses>
@@
 <segment>
 <pinref part="L3" gate="G$1" pin="1"/>
-<wire x1="134.62" y1="195.58" x2="132.08" y2="195.58" width="0.1524" layer="91"/>
+<wire x1="134.62" y1="198.12" x2="132.08" y2="195.58" width="0.1524" layer="91"/>
 <pinref part="SJ2" gate="1" pin="2"/>
 <wire x1="132.08" y1="195.58" x2="127" y2="195.58" width="0.1524" layer="91"/>
@@
 </segment>
 <segment>
-<pinref part="X1" gate="G$1" pin="VCC"/>
-<pinref part="+3V11" gate="G$1" pin="+3V3"/>
-<pinref part="C41" gate="G$1" pin="2"/>
-<wire x1="673.1" y1="170.18" x2="688.34" y2="170.18" width="0.1524" layer="91"/>
-<junction x="673.1" y="170.18"/>
-</segment>
-<segment>
 <pinref part="R29" gate="G$1" pin="1"/>
 <pinref part="+3V12" gate="G$1" pin="+3V3"/>
@@
 <junction x="314.96" y="226.06"/>
 </segment>
+<segment>
+<pinref part="+3V11" gate="G$1" pin="+3V3"/>
+<pinref part="R13" gate="G$1" pin="1"/>
+<wire x1="657.86" y1="170.18" x2="660.4" y2="170.18" width="0.1524" layer="91"/>
+<pinref part="TP11" gate="G$1" pin="TP"/>
+<junction x="660.4" y="170.18"/>
+</segment>
 </net>
 <net name="USB_ID" class="0">
@@
 <pinref part="J1" gate="G$1" pin="VBUS"/>
 <pinref part="L2" gate="G$1" pin="1"/>
-<wire x1="193.04" y1="121.92" x2="198.12" y2="121.92" width="0.1524" layer="91"/>
+<wire x1="193.04" y1="121.92" x2="198.12" y2="124.46" width="0.1524" layer="91"/>
 </segment>
 </net>
@@
 <junction x="231.14" y="121.92"/>
 <pinref part="L2" gate="G$1" pin="2"/>
-<wire x1="208.28" y1="121.92" x2="231.14" y2="121.92" width="0.1524" layer="91"/>
+<wire x1="208.28" y1="124.46" x2="231.14" y2="121.92" width="0.1524" layer="91"/>
 </segment>
 <segment>
@@
 <junction x="152.4" y="195.58"/>
 <pinref part="L3" gate="G$1" pin="2"/>
-<wire x1="152.4" y1="195.58" x2="144.78" y2="195.58" width="0.1524" layer="91"/>
+<wire x1="152.4" y1="195.58" x2="144.78" y2="198.12" width="0.1524" layer="91"/>
 <pinref part="IC3" gate="_PWR" pin="VREF+"/>
 <wire x1="165.1" y1="195.58" x2="162.56" y2="195.58" width="0.1524" layer="91"/>
@@
 </segment>
 </net>
+<net name="VCC" class="0">
+<segment>
+<pinref part="R13" gate="G$1" pin="2"/>
+<pinref part="X1" gate="G$1" pin="VCC"/>
+<wire x1="670.56" y1="170.18" x2="673.1" y2="170.18" width="0.1524" layer="91"/>
+<pinref part="C41" gate="G$1" pin="2"/>
+<wire x1="688.34" y1="170.18" x2="673.1" y2="170.18" width="0.1524" layer="91"/>
+<junction x="673.1" y="170.18"/>
+<pinref part="TP14" gate="G$1" pin="TP"/>
+</segment>
+</net>
