File: Mk3 Prototype.sch (EAGLE design)
At the start: 193 parts, among them IC1 BD49XXX, IC2 NCP1529MU, IC3 STM32F401V, IC4 CC3100, IC5 S25FL216K0PMFI011, J1 ZX62-AB-5PA(11), J2 SFV30R-2STE1HLF, J3 SWD_SHROUD, Q1 DMMT5401, Q2 NTR4101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

Commit message: moving parts around a little
Parts:
- SV2, SV3, SV4, SV5, SV6: device con-lstb:MA03-1 -> TiLDA Mk3 Parts:M03PTH
Other:
- moved on the sheet: SV2, SV3, SV4, SV5, SV6
Changed lines of the file:
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@@
 <part name="C34" library="TiLDA Mk3 Parts" deviceset="C-EU" device="C0402-SMALLER" value="0402/100n/10V/X5R"/>
 <part name="U2" library="TiLDA Mk3 Parts" deviceset="ARDUINOR3" device="-NODIM"/>
-<part name="SV2" library="con-lstb" deviceset="MA03-1" device=""/>
+<part name="SV2" library="TiLDA Mk3 Parts" deviceset="M03" device="PTH"/>
 <part name="D1" library="SparkFun-LED" deviceset="WS2812B" device=""/>
 <part name="GND50" library="TiLDA Mk3 Parts" deviceset="GND" device=""/>
 <part name="GND63" library="TiLDA Mk3 Parts" deviceset="GND" device=""/>
-<part name="SV4" library="con-lstb" deviceset="MA03-1" device=""/>
-<part name="SV6" library="con-lstb" deviceset="MA03-1" device=""/>
-<part name="SV3" library="con-lstb" deviceset="MA03-1" device=""/>
-<part name="SV5" library="con-lstb" deviceset="MA03-1" device=""/>
+<part name="SV4" library="TiLDA Mk3 Parts" deviceset="M03" device="PTH"/>
+<part name="SV6" library="TiLDA Mk3 Parts" deviceset="M03" device="PTH"/>
+<part name="SV3" library="TiLDA Mk3 Parts" deviceset="M03" device="PTH"/>
+<part name="SV5" library="TiLDA Mk3 Parts" deviceset="M03" device="PTH"/>
 <part name="GND64" library="TiLDA Mk3 Parts" deviceset="GND" device=""/>
 <part name="GND66" library="TiLDA Mk3 Parts" deviceset="GND" device=""/>

Commit message: first prototype pretty much done
Parts:
- added ANT2: CHIPANT, TiLDA Mk3 Parts:CHIPANT
- JP4: value M10SILK_FEMALE_PTH -> M10NOSILK; device SparkFun-Connectors:M10SILK_FEMALE_PTH -> TiLDA Mk3 Parts:M10NOSILK
- SV1: device con-lstb:MA03-1 -> TiLDA Mk3 Parts:M03PTH
Connections:
- net ANT: now also ANT2.1; no longer ANT1.SIGNAL
Other:
- note added: "2148522"
- moved on the sheet: SV1
Changed lines of the file:
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@@
 <part name="R38" library="TiLDA Mk3 Parts" deviceset="R-EU_" device="R0402-SMALLER" value="0402/100K/5%"/>
 <part name="GND42" library="TiLDA Mk3 Parts" deviceset="GND" device=""/>
-<part name="GND43" library="TiLDA Mk3 Parts" deviceset="GND" device=""/>
 <part name="R28" library="TiLDA Mk3 Parts" deviceset="R-EU_" device="R0402-SMALLER" value="0402/100K/5%"/>
 <part name="GND44" library="TiLDA Mk3 Parts" deviceset="GND" device=""/>
@@
 <part name="GND85" library="TiLDA Mk3 Parts" deviceset="GND" device=""/>
 <part name="R24" library="TiLDA Mk3 Parts" deviceset="R-EU_" device="R0402-SMALLER" value="0"/>
-<part name="SV1" library="con-lstb" deviceset="MA03-1" device=""/>
+<part name="SV1" library="TiLDA Mk3 Parts" deviceset="M03" device="PTH"/>
 <part name="S6" library="SparkFun-Electromechanical" deviceset="SWITCH-MOMENTARY-2" device="SMD-1101NE"/>
 <part name="GND86" library="TiLDA Mk3 Parts" deviceset="GND" device=""/>
@@
 <part name="D2" library="TiLDA Mk3 Parts" deviceset="DIODE" device="SOD-323F"/>
 <part name="SJ1" library="SparkFun-Passives" deviceset="JUMPER-PAD-2-NO" device="YES_SILK"/>
-<part name="JP4" library="SparkFun-Connectors" deviceset="M10" device="SILK_FEMALE_PTH"/>
+<part name="JP4" library="TiLDA Mk3 Parts" deviceset="M10" device="NOSILK"/>
 <part name="X6" library="con-coax" deviceset="MC-921" device=""/>
 <part name="R41" library="TiLDA Mk3 Parts" deviceset="R-EU_" device="R0402-SMALLER" value="DNP (0ohm)"/>
@@
 <part name="TP11" library="TiLDA Mk3 Parts" deviceset="TP" device="B1,27"/>
 <part name="TP14" library="TiLDA Mk3 Parts" deviceset="TP" device="B1,27"/>
+<part name="ANT2" library="TiLDA Mk3 Parts" deviceset="CHIPANT" device=""/>
 </parts>
 <sheets>
@@
 when screen power is off</text>
 <text x="378.46" y="60.96" size="1.778" layer="91" rot="R90">RETHINK</text>
+<text x="731.52" y="248.92" size="1.778" layer="91">2148522</text>
 </plain>
 <instances>
@@
 <instance part="R38" gate="G$1" x="779.78" y="86.36" rot="R270"/>
 <instance part="GND42" gate="1" x="779.78" y="38.1"/>
-<instance part="GND43" gate="1" x="754.38" y="236.22"/>
 <instance part="R28" gate="G$1" x="764.54" y="58.42" rot="R270"/>
 <instance part="GND44" gate="1" x="764.54" y="35.56"/>
@@
 <attribute name="NAME" x="671.83" y="173.99" size="1.778" layer="95"/>
 </instance>
+<instance part="ANT2" gate="G$1" x="736.6" y="243.84"/>
 </instances>
 <busses>
@@
 <wire x1="736.6" y1="241.3" x2="736.6" y2="238.76" width="0.1524" layer="91"/>
 <junction x="736.6" y="241.3"/>
-<wire x1="736.6" y1="241.3" x2="749.3" y2="241.3" width="0.1524" layer="91"/>
-<wire x1="749.3" y1="241.3" x2="754.38" y2="241.3" width="0.1524" layer="91"/>
-<wire x1="754.38" y1="238.76" x2="754.38" y2="241.3" width="0.1524" layer="91"/>
-<pinref part="GND43" gate="1" pin="GND"/>
-<pinref part="ANT1" gate="G$1" pin="SIGNAL"/>
-<junction x="749.3" y="241.3"/>
+<pinref part="ANT2" gate="G$1" pin="1"/>
 </segment>
 </net>

Commit message: schematic tidyied up
Parts:
- removed ANT1: ANTENNA22500AT44M0400, SparkFun-RF:ANTENNA22500AT44M0400
- removed TP7: TP4MM, TiLDA Mk3 Parts:TP4MM
Connections:
- net A5: no longer TP7.TP
Other:
- note added: "/CC3100 UART"
- note added: "ADC Inputs"
- note added: "DONE:"
- note added: "ESP8266"
- note added: "LEDs"
- note added: "MicroSD Card"
- note added: "Port E"
- note added: "Power"
- note added: "Servo / WS2812 Headers"
- note added: "USB OTG"
- note added: "WS2812"
- note removed: "Consider this T-Hole for swd"
- note removed: "RETHINK"
- note removed: "fairly sure this cap should be at least 16V"
- note removed: "keep this crystal footprint just in case"
- note removed: "might need to be connected to a ftdi header for debug"
- note removed: "might want to change footprint"
- note removed: "orginally two caps of value 0603/22u/4V/X5R"
- note removed: "tim2_ch1"
- moved on the sheet: C13, C17, C18, C2, C25, C26, C37, C41, C46, C5, C57, C58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
