File: Mk3 Prototype.brd (EAGLE design)
At the start: 113 x 55.2 mm, 192 parts, among them IC1 BD49XXX, IC2 NCP1529MU, IC3 STM32F401V, IC4 CC3100, IC5 S25FL216K0PMFI011, J1 ZX62-AB-5PA(11), J2 SFV30R-2STE1HLF, J3 SWD_SHROUD, Q1 DMMT5401, Q2 NTR4101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

Commit message: updating some part values
Parts:
- R12, R14: value (none) -> 0402/150/5%
- R2: value (none) -> 0402/220/5%
Changed lines of the file:
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@@
 <attribute name="VALUE" x="76.516" y="3.5795" size="0.4064" layer="27" rot="R180"/>
 </element>
-<element name="R2" library="TiLDA Mk3 Parts" package="R0402-SMALLER" value="" x="65.5" y="3" smashed="yes" rot="MR270">
+<element name="R2" library="TiLDA Mk3 Parts" package="R0402-SMALLER" value="0402/220/5%" x="65.5" y="3" smashed="yes" rot="MR270">
 <attribute name="NAME" x="66.1015" y="2.289" size="0.8128" layer="26" font="vector" ratio="14" rot="MR270"/>
 <attribute name="VALUE" x="66.643" y="4.0795" size="0.4064" layer="28" rot="MR270"/>
@@
 <attribute name="VALUE" x="22.4205" y="13.016" size="0.4064" layer="27" rot="R270"/>
 </element>
-<element name="R12" library="TiLDA Mk3 Parts" package="R0402-SMALLER" value="" x="26.25" y="11.75" smashed="yes" rot="MR90">
+<element name="R12" library="TiLDA Mk3 Parts" package="R0402-SMALLER" value="0402/150/5%" x="26.25" y="11.75" smashed="yes" rot="MR90">
 <attribute name="NAME" x="26.8485" y="10.661" size="0.8128" layer="26" font="vector" ratio="14" rot="MR90"/>
 <attribute name="VALUE" x="25.107" y="10.6705" size="0.4064" layer="28" rot="MR90"/>
 </element>
-<element name="R14" library="TiLDA Mk3 Parts" package="R0402-SMALLER" value="" x="25" y="13" smashed="yes" rot="MR180">
+<element name="R14" library="TiLDA Mk3 Parts" package="R0402-SMALLER" value="0402/150/5%" x="25" y="13" smashed="yes" rot="MR180">
 <attribute name="NAME" x="25.389" y="11.6985" size="0.8128" layer="26" font="vector" ratio="14" rot="MR0"/>
 <attribute name="VALUE" x="23.9205" y="14.143" size="0.4064" layer="28" rot="MR180"/>

Commit message: one part value changed
Parts:
- R24: value 0 -> 0402/0R
Changed lines of the file:
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@@
 <attribute name="NAME" x="13.1015" y="11.589" size="0.8128" layer="26" font="vector" ratio="14" rot="MR270"/>
 </element>
-<element name="R24" library="TiLDA Mk3 Parts" package="R0402-SMALLER" value="0" x="78.7" y="27.4" smashed="yes" rot="MR180">
+<element name="R24" library="TiLDA Mk3 Parts" package="R0402-SMALLER" value="0402/0R" x="78.7" y="27.4" smashed="yes" rot="MR180">
 <attribute name="NAME" x="77.311" y="28.7015" size="0.8128" layer="26" font="vector" ratio="14" rot="MR180"/>
 </element>
