File: Mk3 Prototype2.sch (EAGLE design)
At the start: 195 parts, among them IC1 BD49XXX, IC2 NCP1529MU, IC3 STM32F401V, IC4 CC3100, IC5 S25FL216K0PMFI011, J1 ZX62-AB-5PA(11), J2 SFV30R-2STE1HLF, J3 SWD_SHROUD, J4 ER-TFT022-1, Q1 DMMT5401, Q2 NTR4101, Q3 NTR4101, Q4 NTR4101, Q5 NTR4101, Q6 NTR4101, SW1 JOYSTICK_MINI_MULTICOMP, U1 JHD12864-G13BSW-OUTLINE, U2 ARDUINOR3-NODIM, U3 MCP73831, U4 USD-SOCKETNEW, X1 ESP-07, X2 CRYSTAL-3.2-2.5, X3 ABS07-32.768KHZ-T, X4 DNP - ABS07-32.768KHZ-T, X5 Q24FA20H00396, X6 MC-921

Commit message: more work on v2
Parts:
- removed C51, C52, C53, C54, C57, C58, C59, C60, C63: 0603/1u/16V/X5R, TiLDA Mk3 Parts:C-EUC0603K-SMALL
- removed J2: SFV30R-2STE1HLF, TiLDA Mk3 Parts:JHD12863-G13BSW-CONNECTOR-SFV30R-2STE1HLF
- removed JP4: M10NOSILK, TiLDA Mk3 Parts:M10NOSILK
- removed S1, S2: SWITCH-MOMENTARY-2, Mine:SWITCH-MOMENTARY-2
- removed U1: JHD12864-G13BSW-OUTLINE, TiLDA Mk3 Parts:JHD12864-G13BSW-OUTLINE
- removed U2: ARDUINOR3-NODIM, TiLDA Mk3 Parts:ARDUINOR3-NODIM
- added ANT1: CHIPANT, TiLDA Mk3 Parts:CHIPANT
- added C38: 0402/4u7/6.3V/X5R, TiLDA Mk3 Parts:C-EUC0402-SMALLER
- added C45: 0402/100n/10V/X5R, TiLDA Mk3 Parts:C-EUC0402-SMALLER
- added IC6: CC3100MOD, TiLDA Mk3 Parts:CC3100MOD
- added JP1, JP2: M10NOSILK, TiLDA Mk3 Parts:M10NOSILK
- added R17: 0402/10K/5%, TiLDA Mk3 Parts:R-EU_R0402-SMALLER
- added R20: 0402/100K/5%, TiLDA Mk3 Parts:R-EU_R0402-SMALLER
- added R47, R48, R49: (no value), TiLDA Mk3 Parts:R-EU_R0402-SMALLER
- added S8: SWITCH-MOMENTARY-2SMD-1101NE, SparkFun-Electromechanical:SWITCH-MOMENTARY-2SMD-1101NE
- added SV7: (no value), TiLDA Mk3 Parts:M03PTH
Connections:
- removed net D2: IC3_PD.PD1, U2.D2
- removed net D4: IC3_PD.PD4, U2.D4
- removed net D7: IC3_PD.PD0, U2.D7
- removed net D8: IC3_PE.PE0, JP4.1, U2.D8
- removed net ESP_GPIO0: IC3_PC.PC1, X1.GPIO0
- removed net ESP_GPIO16: IC3_PC.PC2, X1.GPIO16
- removed net LCD_P1+: C57.2, J2.P1+
- removed net LCD_P1-: C57.1, C58.1, J2.P1-
- removed net LCD_P2+: C60.2, J2.P2+
- removed net LCD_P2-: C60.1, J2.P2-
- removed net LCD_P3+: C58.2, J2.P3+
- removed net LCD_V0: C51.2, J2.V0
- removed net LCD_V1: C52.2, J2.V1
- removed net LCD_V2: C63.2, J2.V2
- removed net LCD_V3: C53.2, J2.V3
- removed net LCD_V4: C54.2, J2.V4
- removed net LCD_VOUT: C59.2, J2.VOUT
- removed net MOM_UP: IC3_PE.PE4, S1.1
- removed net N$57: Q3.D, R32.2
- new net CC_HIB: IC3_PC.PC1, IC6.!HIB, X1.GPIO0
- new net CC_IRQ: IC3_PC.PC2, IC6.IRQ, X1.GPIO16
- new net COMMAND: J4.WRX(D/CX)
- new net LCD0: IC3_PE.PE0, J4.DB0
- new net LCD1: IC3_PE.PE1, J4.DB1
- new net LCD2: IC3_PE.PE2, J4.DB2
- new net LCD3: IC3_PE.PE3, J4.DB3
- new net LCD4: IC3_PE.PE4, J4.DB4
- new net LCD5: IC3_PE.PE5, J4.DB5
- new net LCD6: IC3_PE.PE6, J4.DB6
- new net LCD7: IC3_PE.PE7, J4.DB7
- new net N$14: J4.LEDA, Q3.D
- new net N$36: ANT1.1, IC6.RF_BG
- new net N$41: IC6.SOP2, R17.1
- new net N$43: IC6.RESERVED, R20.1
- new net N$46: J4.LEDK1, R47.2
- new net N$47: J4.LEDK2, R48.2
- new net N$49: J4.LEDK3, R49.2
- new net N$50: IC3_PD.PD1
- new net N$58: IC6.UART1_TX, SV7.3
- new net N$59: IC6.UART1_RX, SV7.2
- new net N$70: J4.IM1, J4.IM2, J4.IM3
- new net SPI3_MISO: J4.SDO
- new net TEAR: J4.TE
- net +3V3: now also C38.2, C45.2, IC6.VBAT_DCDC_ANA, IC6.VBAT_DCDC_DIG, IC6.VBAT_DCDC_PA, J4.VCI, J4.VDDI; no longer S1.2, S2.1, U2.3V, U2.IOREF
- net A0: no longer U2.A0
- net A1: no longer U2.A1
- net A2: no longer U2.A2
- net A3: no longer U2.A3
- net A4: no longer U2.A4/SDA
- net A5: no longer U2.A5/SCL
- net AREF: no longer JP4.8, U2.AREF
- net ESP_CH_PD: now also IC6.!RESET, S8.1
- net GND: now also C38.1, C45.1, IC6.GND, J4.DB10, J4.DB11, J4.DB12, J4.DB13, J4.DB14, J4.DB15, J4.DB16, J4.DB17, J4.DB8, J4.DB9, J4.DE, J4.DOTCLK, J4.GND, J4.HSYNC, J4.IM0, J4.VSYNC, R17.2, R20.2, R47.1, R48.1, R49.1, S8.2, SV7.1; no longer C51.1, C52.1, C53.1, C54.1, C59.1, C63.1, J2.PS, J2.VSS, JP4.7, U1.K, U2.GND, U2.GND1, U2.GND2
- net I2C_SCL: no longer JP4.10, U2.SCL
- net I2C_SDA: no longer JP4.9, U2.SDA
- net LCD_!RST: now also J4.RESET; no longer IC3_PE.PE1, J2.RST
- net LCD_A0: no longer J2.A0
- net LCD_POWER: no longer IC3_PB.PB4
- net LCD_VCC: no longer J2.C86, J2.D0, J2.D1, J2.D2, J2.D3, J2.D4, J2.D5, J2.RD, J2.VDD, J2.WR
- net MCO1: no longer IC3_PA.PA8
- net MOM_LEFT: no longer S2.2
- net MOM_RIGHT: no longer IC3_PE.PE7
- net N$1: now also IC3_PD.PD0; no longer R32.1, U1.A
- net NRST: no longer U2./RESET
- net SPI1_MISO: now also IC6.SPI_DOUT; no longer IC4_HOST_SPI.MISO
- net SPI1_MOSI: now also IC6.SPI_DIN; no longer IC4_HOST_SPI.MOSI
- net SPI1_NSS: now also IC6.!SPI_CS; no longer IC4_HOST_SPI.!CS
- net SPI1_SCK: now also IC6.SPI_CLK; no longer IC4_HOST_SPI.CLK
- net SPI2_CLK: no longer JP4.6, U2.D13
- net SPI2_MISO: no longer JP4.5, U2.D12
- net SPI2_MOSI: no longer JP4.4, U2.D11
- net SPI3_MOSI: now also J4.SDI; no longer J2.D7
- net SPI3_NSS: now also J4.CSX; no longer J2.CS1B
- net SPI3_SCK: now also J4.D/CX(SCL); no longer J2.D6
- net SPI4_MOSI: no longer IC3_PE.PE6
- net TIM10_CH1: no longer JP4.2, U2.D9
- net TIM11_CH1: no longer JP4.3, U2.D10
- net TIM1_CH1N: no longer U2.D3
- net TIM4_CH2: no longer U2.D5
- net TIM4_CH3: no longer U2.D6
- net TIM9_CH1: no longer IC3_PE.PE5
- net USART2_RX: now also R46.1, X1.UTXD; no longer TP1.TP, U2.D0
- net USART2_TX: now also IC4_UART.RX, SV1.2, X1.URXD; no longer TP2.TP, U2.D1
- net USART6_RX: now also TP1.TP; no longer R46.1, X1.UTXD
- net USART6_TX: now also TP2.TP; no longer IC4_UART.RX, SV1.2, X1.URXD
- net VBUS: no longer U2.5V, U2.VIN
- net WIFI_INTR: no longer IC3_PE.PE3
Other:
- note added: "0: parallel; 1: serial"
- note added: "5 ohm"
- note added: "add footprint for cap"
- note added: "lcd_!RST"
- note added: "mom_right"
- note added: "mom_up"
- note added: "spi4_mosi"
- note added: "tim9_ch1"
- note added: "wifi_inter"
- note removed: "USB AB Socket"
- moved on the sheet: Q3

Commit message: initial schematic of v2 done
Connections:
- net MOM_LEFT renamed BOOT1
- removed net A0: IC3_PA.PA1
- removed net A1: IC3_PA.PA2
- removed net A2: IC3_PC.PC4
- removed net A3: IC3_PC.PC5
- removed net I2C_SCL: IC3_PB.PB6
- removed net I2C_SDA: IC3_PB.PB7
- removed net LCD_A0: IC3_PD.PD7
- removed net N$1: IC3_PD.PD0
- removed net N$50: IC3_PD.PD1
- removed net N$70: J4.IM1, J4.IM2, J4.IM3
- removed net SPI4_MOSI: D1.DIN
- new net BTN_MENU: IC3_PD.PD1, S7.2
- new net LCD_ADC_X: IC3_PC.PC0, J4.X-
- new net LCD_ADC_Y: IC3_PC.PC1, J4.Y-
- new net LCD_MODE: IC3_PB.PB6, J4.IM1, J4.IM2, J4.IM3
- new net LCD_RD: IC3_PD.PD4, J4.RD
- new net LCD_X: IC3_PC.PC3, J4.X+
- new net LCD_Y: IC3_PC.PC13, J4.Y+
- new net SPI2_NSS: IC3_PB.PB12, JP2.7
- new net TIM2_CH1: IC3_PA.PA0, JP1.7
- new net TIM2_CH2: IC3_PA.PA1, JP1.8
- new net TIM2_CH3: IC3_PA.PA2, JP1.9
- new net TIM2_CH4: IC3_PA.PA3, JP1.10
- net A4: no longer IC3_PB.PB0
- net ADC_LIGHT: no longer IC3_PA.PA3
- net ADC_VBUS: no longer IC3_PA.PA0
- net ADC_VIN: now also IC3_PB.PB0; no longer IC3_PC.PC3
- net CC_HIB: now also IC3_PC.PC5; no longer IC3_PC.PC1
- net COMMAND: now also IC3_PD.PD7
- net ESP_CH_PD: now also IC3_PC.PC4; no longer IC3_PC.PC0
- net LCD_!RST: now also IC3_PB.PB7
- net LED2: now also IC3_PE.PE12; no longer IC3_PB.PB10
- net MOM_RIGHT: now also IC3_PD.PD0
- net SPI2_CLK: now also IC3_PB.PB10, JP2.8; no longer IC3_PD.PD3
- net SPI2_MISO: now also JP2.9
- net SPI2_MOSI: now also JP2.10
- net SPI3_MISO: now also IC3_PB.PB4
- net TEAR: now also IC3_PD.PD3
- net TIM10_CH1: now also JP1.5
- net TIM11_CH1: now also JP1.6
- net TIM1_CH1: now also JP2.1
- net TIM1_CH2: now also JP2.2
- net TIM1_CH3: now also JP2.3
- net TIM1_CH4: now also D1.DIN, JP2.4
- net USART6_RX: now also JP2.6
- net USART6_TX: now also JP2.5
- net WIFI_!HIB: no longer IC3_PC.PC13
Other:
- note added: "adc_light"
- note added: "adc_vbus"
- note added: "extra backlight connection if 2.4""
- note added: "i2c"
- note added: "is 3.3V fine?"
- note added: "led2"
- note removed: "lcd_!RST"
- note removed: "mom_right"
- note removed: "mom_up"
- note removed: "tim9_ch1"
- note removed: "wifi_inter"
- moved on the sheet: C38, C45, JP1, JP2

Commit message: more schematic stuff
Parts:
- removed Q4: NTR4101, TiLDA Mk3 Parts:MOSFET-P-SOT23
- removed R44: 0402/1R/5%, TiLDA Mk3 Parts:R-EU_R0402-SMALLER
- removed TP12, TP13: TPB1,27, TiLDA Mk3 Parts:TPB1,27
Connections:
- removed net BOOT1: IC3_PB.PB2, R11.2
- removed net LCD_POWER: Q4.G
- removed net LCD_VCC: Q4.D
- removed net N$53: Q4.S, R44.2, TP13.TP
- net +3V3: no longer R44.1, TP12.TP
- net A5: no longer IC3_PB.PB1
- net ADC_LIGHT: now also IC3_PB.PB1
- net ADC_VBUS: now also IC3_PC.PC4
- net COMMAND: now also IC3_PB.PB7; no longer IC3_PD.PD7
- net ESP_CH_PD: now also IC3_PB.PB2, R11.2; no longer IC3_PC.PC4
- net LCD_!RST: now also IC3_PD.PD7; no longer IC3_PB.PB7
- net LCD_MODE: now also IC3_PD.PD4; no longer IC3_PB.PB6
- net LCD_RD: now also IC3_PB.PB6; no longer IC3_PD.PD4
- net WIFI_!RESET: no longer IC3_PE.PE8
Other:
- note added: "add small resistors to stop shorting agaoinst vcc/gnd"
- note added: "unconnected"
- note removed: "adc_light"
- note removed: "adc_vbus"
- note removed: "spi4_mosi"
Changed lines of the file:
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@@
 <part name="IC2" library="TiLDA Mk3 Parts" deviceset="NCP1529" device="MU"/>
 <part name="R43" library="TiLDA Mk3 Parts" deviceset="R-EU_" device="R0402-SMALLER" value="0402/220/5%"/>
-<part name="R44" library="TiLDA Mk3 Parts" deviceset="R-EU_" device="R0402-SMALLER" value="0402/1R/5%"/>
-<part name="Q4" library="TiLDA Mk3 Parts" deviceset="MOSFET-P" device="-SOT23" value="NTR4101"/>
 <part name="Q6" library="TiLDA Mk3 Parts" deviceset="MOSFET-P" device="-SOT23" value="NTR4101"/>
 <part name="R45" library="TiLDA Mk3 Parts" deviceset="R-EU_" device="R0402-SMALLER" value="0402/220k/5%"/>
@@
 <part name="C27" library="passives-7351" deviceset="CAPACITOR" device="0805-N" value="0805/22u/??V/X5R"/>
 <part name="C40" library="passives-7351" deviceset="CAPACITOR" device="0805-N" value="0805/22u/??V/X5R"/>
-<part name="TP12" library="TiLDA Mk3 Parts" deviceset="TP" device="B1,27"/>
-<part name="TP13" library="TiLDA Mk3 Parts" deviceset="TP" device="B1,27"/>
 <part name="R46" library="TiLDA Mk3 Parts" deviceset="R-EU_" device="R0402-SMALLER" value="0402/10K/5%"/>
 <part name="R13" library="TiLDA Mk3 Parts" deviceset="R-EU_" device="R0402-SMALLER" value="0402/0.1R/5%"/>
@@
 <text x="322.58" y="383.54" size="1.778" layer="91">0: parallel; 1: serial</text>
 <text x="347.98" y="393.7" size="1.778" layer="91">5 ohm</text>
-<text x="91.44" y="55.88" size="1.778" layer="91">spi4_mosi</text>
 <text x="81.28" y="175.26" size="1.778" layer="91">led2</text>
-<text x="-7.62" y="203.2" size="1.778" layer="91">adc_vbus</text>
-<text x="-7.62" y="198.12" size="1.778" layer="91">adc_light</text>
 <text x="337.82" y="78.74" size="1.778" layer="91">i2c</text>
 <text x="337.82" y="76.2" size="1.778" layer="91">i2c</text>
 <text x="363.22" y="393.7" size="1.778" layer="91">extra backlight connection if 2.4"</text>
 <text x="322.58" y="292.1" size="1.778" layer="91">is 3.3V fine?</text>
+<text x="58.42" y="48.26" size="1.778" layer="91">unconnected</text>
+<text x="596.9" y="170.18" size="1.778" layer="91">add small resistors to stop shorting agaoinst vcc/gnd</text>
 </plain>
 <instances>
@@
 <attribute name="VALUE" x="29.21" y="227.838" size="1.778" layer="96"/>
 </instance>
-<instance part="R44" gate="G$1" x="317.5" y="226.06"/>
-<instance part="Q4" gate="G$1" x="335.28" y="226.06" rot="R90"/>
 <instance part="Q6" gate="G$1" x="642.62" y="58.42" rot="R90"/>
 <instance part="R45" gate="G$1" x="635" y="50.8" rot="R270"/>
@@
 <attribute name="VALUE" x="444.881" y="205.74" size="1.778" layer="96" rot="R270"/>
 </instance>
-<instance part="TP12" gate="G$1" x="312.42" y="231.14" smashed="yes">
-<attribute name="NAME" x="311.15" y="232.41" size="1.778" layer="95"/>
-</instance>
-<instance part="TP13" gate="G$1" x="322.58" y="231.14" smashed="yes">
-<attribute name="NAME" x="321.31" y="232.41" size="1.778" layer="95"/>
-</instance>
 <instance part="R46" gate="G$1" x="208.28" y="88.9" smashed="yes" rot="R90">
 <attribute name="NAME" x="206.7814" y="85.09" size="1.778" layer="95" rot="R90"/>
@@
 </segment>
 <segment>
-<wire x1="71.12" y1="200.66" x2="68.58" y2="200.66" width="0.1524" layer="91"/>
-<label x="71.12" y="200.66" size="1.778" layer="95"/>
-<pinref part="IC3" gate="_PB" pin="PB1"/>
-</segment>
-<segment>
 <wire x1="617.22" y1="137.16" x2="617.22" y2="147.32" width="0.1524" layer="91"/>
 <label x="617.22" y="137.16" size="1.778" layer="95" rot="R90"/>
@@
 <wire x1="332.74" y1="218.44" x2="332.74" y2="220.98" width="0.1524" layer="91"/>
 <label x="312.42" y="218.44" size="1.778" layer="95"/>
-<pinref part="Q4" gate="G$1" pin="G"/>
 </segment>
 </net>
@@
 </segment>
 <segment>
-<pinref part="IC3" gate="_PB" pin="PB7"/>
-<wire x1="68.58" y1="185.42" x2="71.12" y2="185.42" width="0.1524" layer="91"/>
-<label x="71.12" y="185.42" size="1.778" layer="95"/>
+<pinref part="IC3" gate="_PD" pin="PD7"/>
+<wire x1="73.66" y1="116.84" x2="83.82" y2="116.84" width="0.1524" layer="91"/>
+<label x="76.2" y="116.84" size="1.778" layer="95"/>
 </segment>
 </net>
@@
 <pinref part="S6" gate="G$1" pin="1"/>
 </segment>
-<segment>
-<pinref part="IC3" gate="_PE" pin="PE8"/>
-<wire x1="73.66" y1="48.26" x2="78.74" y2="48.26" width="0.1524" layer="91"/>
-<label x="76.2" y="48.26" size="1.778" layer="95"/>
-</segment>
 </net>
 <net name="WIFI_FORCE_AP" class="0">
@@
 </segment>
 <segment>
-<pinref part="R44" gate="G$1" pin="1"/>
 <pinref part="+3V9" gate="G$1" pin="+3V3"/>
-<pinref part="TP12" gate="G$1" pin="TP"/>
 <wire x1="312.42" y1="228.6" x2="312.42" y2="226.06" width="0.1524" layer="91"/>
 <wire x1="307.34" y1="226.06" x2="312.42" y2="226.06" width="0.1524" layer="91"/>
-<junction x="312.42" y="226.06"/>
 </segment>
 <segment>
@@
 <wire x1="508" y1="33.02" x2="515.62" y2="33.02" width="0.1524" layer="91"/>
 </segment>
+<segment>
+<pinref part="IC3" gate="_PC" pin="PC4"/>
+<wire x1="33.02" y1="124.46" x2="35.56" y2="124.46" width="0.1524" layer="91"/>
+<label x="35.56" y="124.46" size="1.778" layer="95"/>
+</segment>
 </net>
 <net name="MCO1" class="0">
@@
 <wire x1="149.86" y1="43.18" x2="149.86" y2="45.72" width="0.1524" layer="91"/>
 </segment>
+<segment>
+<pinref part="IC3" gate="_PB" pin="PB1"/>
+<wire x1="68.58" y1="200.66" x2="71.12" y2="200.66" width="0.1524" layer="91"/>
+<label x="71.12" y="200.66" size="1.778" layer="95"/>
+</segment>
 </net>
 <net name="ESP_CH_PD" class="0">
@@
 </segment>
 <segment>
-<pinref part="IC3" gate="_PC" pin="PC4"/>
-<wire x1="33.02" y1="124.46" x2="35.56" y2="124.46" width="0.1524" layer="91"/>
-<label x="35.56" y="124.46" size="1.778" layer="95"/>
+<pinref part="IC3" gate="_PB" pin="PB2"/>
+<label x="71.12" y="198.12" size="1.778" layer="95"/>
+<pinref part="R11" gate="G$1" pin="2"/>
+<wire x1="68.58" y1="198.12" x2="88.9" y2="198.12" width="0.1524" layer="91"/>
+<junction x="88.9" y="198.12"/>
+<wire x1="88.9" y1="198.12" x2="93.98" y2="198.12" width="0.1524" layer="91"/>
 </segment>
 </net>
@@
 <net name="N$53" class="0">
 <segment>
-<pinref part="R44" gate="G$1" pin="2"/>
-<pinref part="Q4" gate="G$1" pin="S"/>
-<pinref part="TP13" gate="G$1" pin="TP"/>
 <wire x1="322.58" y1="228.6" x2="322.58" y2="226.06" width="0.1524" layer="91"/>
 <wire x1="322.58" y1="226.06" x2="330.2" y2="226.06" width="0.1524" layer="91"/>
-<junction x="322.58" y="226.06"/>
 </segment>
 </net>
@@
 <junction x="360.68" y="220.98"/>
 <wire x1="340.36" y1="226.06" x2="360.68" y2="226.06" width="0.1524" layer="91"/>
-<pinref part="Q4" gate="G$1" pin="D"/>
 </segment>
 </net>
@@
 </segment>
 <segment>
-<pinref part="IC3" gate="_PD" pin="PD7"/>
-<wire x1="73.66" y1="116.84" x2="83.82" y2="116.84" width="0.1524" layer="91"/>
-<label x="76.2" y="116.84" size="1.778" layer="95"/>
+<pinref part="IC3" gate="_PB" pin="PB7"/>
+<wire x1="68.58" y1="185.42" x2="71.12" y2="185.42" width="0.1524" layer="91"/>
+<label x="71.12" y="185.42" size="1.778" layer="95"/>
 </segment>
 </net>
@@
 </segment>
 <segment>
-<pinref part="IC3" gate="_PD" pin="PD4"/>
-<wire x1="73.66" y1="124.46" x2="83.82" y2="124.46" width="0.1524" layer="91"/>
-<label x="76.2" y="124.46" size="1.778" layer="95"/>
+<pinref part="IC3" gate="_PB" pin="PB6"/>
+<wire x1="68.58" y1="187.96" x2="71.12" y2="187.96" width="0.1524" layer="91"/>
+<label x="71.12" y="187.96" size="1.778" layer="95"/>
 </segment>
 </net>
@@
 <net name="LCD_MODE" class="0">
 <segment>
-<pinref part="IC3" gate="_PB" pin="PB6"/>
-<wire x1="68.58" y1="187.96" x2="71.12" y2="187.96" width="0.1524" layer="91"/>
-<label x="71.12" y="187.96" size="1.778" layer="95"/>
-</segment>
-<segment>
 <pinref part="J4" gate="G$1" pin="IM1"/>
 <wire x1="355.6" y1="388.62" x2="358.14" y2="388.62" width="0.1524" layer="91"/>
@@
 <junction x="355.6" y="383.54"/>
 </segment>
+<segment>
+<pinref part="IC3" gate="_PD" pin="PD4"/>
+<wire x1="73.66" y1="124.46" x2="83.82" y2="124.46" width="0.1524" layer="91"/>
+<label x="76.2" y="124.46" size="1.778" layer="95"/>
+</segment>
 </net>
 <net name="LCD_ADC_X" class="0">
@@
 </segment>
 </net>
-<net name="BOOT1" class="0">
-<segment>
-<pinref part="IC3" gate="_PB" pin="PB2"/>
-<label x="71.12" y="198.12" size="1.778" layer="95"/>
-<pinref part="R11" gate="G$1" pin="2"/>
-<wire x1="68.58" y1="198.12" x2="88.9" y2="198.12" width="0.1524" layer="91"/>
-<junction x="88.9" y="198.12"/>
-<wire x1="88.9" y1="198.12" x2="93.98" y2="198.12" width="0.1524" layer="91"/>
-</segment>
-</net>

Commit message: moving parts around a bit
Parts:
- removed G1: GND-LOOP, dtb:GND-LOOP
Connections:
- net GND: no longer G1.1, G1.2
Changed lines of the file:
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@@
 <part name="GND79" library="TiLDA Mk3 Parts" deviceset="GND" device=""/>
 <part name="L3" library="TiLDA Mk3 Parts" deviceset="WE-CBF" device="_0805" value="Bead"/>
-<part name="G1" library="dtb" deviceset="GND-LOOP" device="" value="GND-LOOP"/>
-<part name="GND56" library="TiLDA Mk3 Parts" deviceset="GND" device=""/>
-<part name="GND57" library="TiLDA Mk3 Parts" deviceset="GND" device=""/>
 <part name="IC3" library="TiLDA Mk3 Parts" deviceset="STM32F401V" device=""/>
 <part name="C29" library="TiLDA Mk3 Parts" deviceset="C-EU" device="C0402-SMALLER" value="0402/2.2u/6.3V/X5R"/>
@@
 <instance part="GND79" gate="1" x="254" y="177.8"/>
 <instance part="L3" gate="G$1" x="139.7" y="193.04"/>
-<instance part="G1" gate="G$1" x="673.1" y="17.78"/>
-<instance part="GND56" gate="1" x="670.56" y="10.16"/>
-<instance part="GND57" gate="1" x="675.64" y="10.16"/>
 <instance part="IC3" gate="_PD" x="68.58" y="114.3"/>
 <instance part="IC3" gate="_PE" x="66.04" y="50.8"/>
@@
 </segment>
 <segment>
-<pinref part="G1" gate="G$1" pin="1"/>
-<pinref part="GND56" gate="1" pin="GND"/>
-</segment>
-<segment>
-<pinref part="G1" gate="G$1" pin="2"/>
-<pinref part="GND57" gate="1" pin="GND"/>
-</segment>
-<segment>

Commit message: changing to 2.4 screen, 0603 componments
Parts:
- removed J4: ER-TFT022-1, TiLDA Mk3 Parts:ER-TFT022-1
- added J2: ER-TFT024-3, TiLDA Mk3 Parts:ER-TFT024-3
- added R44: (no value), TiLDA Mk3 Parts:R-EU_0603K-SMALL
- C10, C11, C12, C13, C14, C15, C16, C18, C19, C20, C21, C22, C23, C24, C29, C33, C34, C38, C39, C8, C9: device TiLDA Mk3 Parts:C-EUC0402-SMALLER -> TiLDA Mk3 Parts:C-EUC0603K-SMALL
- R1: device TiLDA Mk3 Parts:R-EU_0207/10 -> TiLDA Mk3 Parts:R-EU_0603K-SMALL
- R10, R11, R12, R14, R15, R16, R18, R19, R2, R21, R22, R23, R25, R3, R33, R4, R43, R45, R47, R48, R49, R5, R6, R7, R8, R9: device TiLDA Mk3 Parts:R-EU_R0402-SMALLER -> TiLDA Mk3 Parts:R-EU_0603K-SMALL
Connections:
- new net N$1: J2.LEDK4, R44.2
- net +3V3: now also J2.VCI, J2.VDDI; no longer J4.VCI, J4.VDDI
- net COMMAND: now also J2.WRX(D/CX); no longer J4.WRX(D/CX)
- net GND: now also J2.DB10, J2.DB11, J2.DB12, J2.DB13, J2.DB14, J2.DB15, J2.DB16, J2.DB17, J2.DB8, J2.DB9, J2.DE, J2.DOTCLK, J2.GND, J2.HSYNC, J2.IM0, J2.VSYNC, R44.1; no longer J4.DB10, J4.DB11, J4.DB12, J4.DB13, J4.DB14, J4.DB15, J4.DB16, J4.DB17, J4.DB8, J4.DB9, J4.DE, J4.DOTCLK, J4.GND, J4.HSYNC, J4.IM0, J4.VSYNC
- net LCD0: now also J2.DB0; no longer J4.DB0
- net LCD1: now also J2.DB1; no longer J4.DB1
- net LCD2: now also J2.DB2; no longer J4.DB2
- net LCD3: now also J2.DB3; no longer J4.DB3
- net LCD4: now also J2.DB4; no longer J4.DB4
- net LCD5: now also J2.DB5; no longer J4.DB5
- net LCD6: now also J2.DB6; no longer J4.DB6
- net LCD7: now also J2.DB7; no longer J4.DB7
- net LCD_!RST: now also J2.RESET; no longer J4.RESET
- net LCD_ADC_X: now also J2.X-; no longer J4.X-
- net LCD_ADC_Y: now also J2.Y-; no longer J4.Y-
- net LCD_MODE: now also J2.IM1, J2.IM2, J2.IM3; no longer J4.IM1, J4.IM2, J4.IM3
- net LCD_RD: now also J2.RD; no longer J4.RD
- net LCD_X: now also J2.X+; no longer J4.X+
- net LCD_Y: now also J2.Y+; no longer J4.Y+
- net N$12: no longer IC2.EN
- net N$14: now also J2.LEDA; no longer J4.LEDA
- net N$46: now also J2.LEDK1; no longer J4.LEDK1
- net N$47: now also J2.LEDK2; no longer J4.LEDK2
- net N$49: now also J2.LEDK3; no longer J4.LEDK3
- net SPI3_MISO: now also J2.SDO; no longer J4.SDO
- net SPI3_MOSI: now also J2.SDI; no longer J4.SDI
- net SPI3_NSS: now also J2.CSX; no longer J4.CSX
- net SPI3_SCK: now also J2.D/CX(SCL); no longer J4.D/CX(SCL)
- net TEAR: now also J2.TE; no longer J4.TE
Other:
- note removed: "extra backlight connection if 2.4""

Commit message: some more routing
Connections:
- net SPI2_CLK: now also JP2.7; no longer JP2.8
- net SPI2_MISO: now also JP2.8; no longer JP2.9
- net SPI2_MOSI: now also JP2.9; no longer JP2.10
- net SPI2_NSS: now also JP2.6; no longer JP2.7
- net TIM10_CH1: now also JP2.2; no longer JP1.5
- net TIM11_CH1: now also JP2.3; no longer JP1.6
- net TIM1_CH1: now also JP1.6; no longer JP2.1
- net TIM1_CH2: now also JP1.7; no longer JP2.2
- net TIM1_CH3: now also JP1.8; no longer JP2.3
- net TIM1_CH4: now also JP1.9; no longer JP2.4
- net TIM2_CH1: now also JP1.2; no longer JP1.7
- net TIM2_CH2: now also JP1.3; no longer JP1.8
- net TIM2_CH3: now also JP1.4; no longer JP1.9
- net TIM2_CH4: now also JP1.5; no longer JP1.10
- net USART6_RX: now also JP2.5; no longer JP2.6
- net USART6_TX: now also JP2.4; no longer JP2.5
Other:
- note added: "Headers"
- note removed: "Arduino Shield Headers"
- moved on the sheet: JP1, JP2
