File: Mk3 Prototype2.sch (EAGLE design)
At the start: 142 parts, among them IC1 TPD3E001DRL, IC2 TPS62082, IC3 STM32F401V, IC4 BQ2409X, IC6 CC3100MOD, IC7 BQ2970, J1 ZX62-AB-5PA(11), J2 ER-TFT024-3, J3 SWD_SHROUD, Q1 DMMT5401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

Commit message: some prodding
Parts:
- added SG1: BUZZER-PKLCS1212E, TiLDA Mk3 Parts:BUZZER-PKLCS1212E
Other:
- note added: "add testpoints"
Changed lines of the file:
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@@
 <part name="R26" library="TiLDA Mk3 Parts" deviceset="R-EU_" device="0603K-SMALL" value="TEmp"/>
 <part name="U1" library="TiLDA Mk3 Parts" deviceset="USD-SOCKET-SDIO" device="DM3AT_0011"/>
+<part name="SG1" library="TiLDA Mk3 Parts" deviceset="BUZZER" device="-PKLCS1212E"/>
 </parts>
 <sheets>
@@
 <text x="414.02" y="50.8" size="1.778" layer="91">change footprint once final part is known</text>
 <text x="693.42" y="160.02" size="1.778" layer="91">connect pin 10</text>
+<text x="693.42" y="154.94" size="1.778" layer="91">add testpoints</text>
 </plain>
 <instances>
@@
 <instance part="R26" gate="G$1" x="40.64" y="99.06"/>
 <instance part="U1" gate="G$1" x="441.96" y="30.48"/>
+<instance part="SG1" gate="G$1" x="223.52" y="60.96"/>
 </instances>
 <busses>

Commit message: cleaning up silk a little
Parts:
- removed SJ3: JUMPER-PAD-2-NOYES_SILK, SparkFun-Passives:JUMPER-PAD-2-NOYES_SILK
- added R27: 0603/220k/5%, TiLDA Mk3 Parts:R-EU_0603K-SMALL
- added TP11: TPB1,27, TiLDA Mk3 Parts:TPB1,27
Connections:
- new net N$17: IC6.FORCE_AP, R27.1, TP11.TP
- net GND: now also R27.2
- net USB_ID: no longer SJ3.1, SJ3.2
Other:
- note added: "orginally 1K, check to see if value is important"
- note removed: "ESD!"
- note removed: "JOY_CENTRE/BOOT0"
- note removed: "needed?"
- moved on the sheet: R20
Changed lines of the file:
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@@
 <attribute name="FARNELL" value="1781089"/>
 </part>
-<part name="SJ3" library="SparkFun-Passives" deviceset="JUMPER-PAD-2-NO" device="YES_SILK"/>
 <part name="R10" library="TiLDA Mk3 Parts" deviceset="R-EU_" device="0603K-SMALL" value="0603/2k/5%"/>
 <part name="Q1" library="TiLDA Mk3 Parts" deviceset="DMMT5401" device="">
@@
 <part name="U1" library="TiLDA Mk3 Parts" deviceset="USD-SOCKET-SDIO" device="DM3AT_0011"/>
 <part name="SG1" library="TiLDA Mk3 Parts" deviceset="BUZZER" device="-PKLCS1212E"/>
+<part name="R27" library="TiLDA Mk3 Parts" deviceset="R-EU_" device="0603K-SMALL" value="0603/220k/5%"/>
+<part name="TP11" library="TiLDA Mk3 Parts" deviceset="TP" device="B1,27"/>
 </parts>
 <sheets>
@@
 <text x="162.56" y="17.78" size="1.778" layer="91" rot="R90">depends on led</text>
 <text x="86.36" y="198.12" size="1.778" layer="91">/ BOOT1</text>
-<text x="160.02" y="132.08" size="1.778" layer="90">ESD!</text>
 <text x="152.146" y="102.87" size="1.778" layer="91">close for OTG</text>
 <text x="358.14" y="127" size="1.778" layer="91">/ JOY_CEN</text>
@@
 <wire x1="246.38" y1="248.92" x2="246.38" y2="254" width="0.1524" layer="97"/>
 <wire x1="246.38" y1="241.3" x2="236.22" y2="241.3" width="0.1524" layer="97"/>
-<text x="-15.24" y="96.52" size="1.778" layer="91">JOY_CENTRE/BOOT0</text>
 <text x="-15.24" y="93.98" size="1.778" layer="91">connect i2c on pb11</text>
 <text x="-15.24" y="91.44" size="1.778" layer="91">speaker to tim1</text>
@@
 <text x="579.12" y="-45.72" size="1.778" layer="91" rot="R90">depends on whether battery has thermistor</text>
 <text x="83.82" y="71.12" size="1.778" layer="91">/JOY_CENTRE</text>
-<text x="162.56" y="106.68" size="1.778" layer="91">needed?</text>
 <text x="414.02" y="50.8" size="1.778" layer="91">change footprint once final part is known</text>
 <text x="693.42" y="160.02" size="1.778" layer="91">connect pin 10</text>
 <text x="693.42" y="154.94" size="1.778" layer="91">add testpoints</text>
+<text x="152.4" y="114.3" size="1.778" layer="91">orginally 1K, check to see if value is important</text>
 </plain>
 <instances>
@@
 <attribute name="FARNELL" x="142.24" y="127" size="1.778" layer="96" display="off"/>
 </instance>
-<instance part="SJ3" gate="G$1" x="154.94" y="109.22" smashed="yes" rot="R180">
-<attribute name="NAME" x="157.48" y="106.68" size="1.778" layer="95" rot="R180"/>
-</instance>
 <instance part="R10" gate="G$1" x="165.1" y="116.84" rot="R180"/>
 <instance part="Q1" gate="G$1" x="612.14" y="43.18">
@@
 <attribute name="FARNELL" x="754.38" y="233.68" size="1.778" layer="96" display="off"/>
 </instance>
-<instance part="GND11" gate="1" x="678.18" y="190.5"/>
+<instance part="GND11" gate="1" x="675.64" y="165.1"/>
 <instance part="R17" gate="G$1" x="736.6" y="157.48" rot="R270"/>
 <instance part="GND43" gate="1" x="736.6" y="149.86"/>
-<instance part="R20" gate="G$1" x="678.18" y="203.2" rot="R270"/>
+<instance part="R20" gate="G$1" x="675.64" y="175.26" rot="R270"/>
 <instance part="+3V26" gate="G$1" x="673.1" y="243.84"/>
 <instance part="SV7" gate="G$1" x="759.46" y="190.5" rot="MR0"/>
@@
 <instance part="U1" gate="G$1" x="441.96" y="30.48"/>
 <instance part="SG1" gate="G$1" x="223.52" y="60.96"/>
+<instance part="R27" gate="G$1" x="673.1" y="175.26" rot="R270"/>
+<instance part="TP11" gate="G$1" x="670.56" y="182.88" smashed="yes" rot="R90">
+<attribute name="NAME" x="669.29" y="181.61" size="1.778" layer="95" rot="R90"/>
+</instance>
 </instances>
 <busses>
@@
 <pinref part="GND11" gate="1" pin="GND"/>
 <pinref part="R20" gate="G$1" pin="2"/>
-<wire x1="678.18" y1="198.12" x2="678.18" y2="193.04" width="0.1524" layer="91"/>
-<junction x="678.18" y="193.04"/>
+<wire x1="675.64" y1="167.64" x2="678.18" y2="167.64" width="0.1524" layer="91"/>
+<wire x1="675.64" y1="170.18" x2="675.64" y2="167.64" width="0.1524" layer="91"/>
+<pinref part="R27" gate="G$1" pin="2"/>
+<wire x1="673.1" y1="170.18" x2="673.1" y2="167.64" width="0.1524" layer="91"/>
+<wire x1="673.1" y1="167.64" x2="675.64" y2="167.64" width="0.1524" layer="91"/>
+<junction x="675.64" y="167.64"/>
 </segment>
 <segment>
@@
 <pinref part="IC6" gate="G$1" pin="RESERVED"/>
 <pinref part="R20" gate="G$1" pin="1"/>
+<wire x1="675.64" y1="180.34" x2="678.18" y2="180.34" width="0.1524" layer="91"/>
 </segment>
 </net>
@@
 <segment>
 <label x="170.18" y="109.22" size="1.778" layer="95"/>
-<wire x1="177.8" y1="109.22" x2="160.02" y2="109.22" width="0.1524" layer="91"/>
-<pinref part="SJ3" gate="G$1" pin="1"/>
-<wire x1="160.02" y1="109.22" x2="160.02" y2="111.76" width="0.1524" layer="91"/>
 <pinref part="J1" gate="G$1" pin="USBID"/>
 <label x="132.08" y="109.22" size="1.778" layer="95"/>
-<pinref part="SJ3" gate="G$1" pin="2"/>
 <wire x1="114.3" y1="121.92" x2="127" y2="121.92" width="0.1524" layer="91"/>
 <wire x1="127" y1="121.92" x2="127" y2="109.22" width="0.1524" layer="91"/>
-<wire x1="127" y1="109.22" x2="149.86" y2="109.22" width="0.1524" layer="91"/>
+<wire x1="127" y1="109.22" x2="177.8" y2="109.22" width="0.1524" layer="91"/>
 <junction x="127" y="109.22"/>
 <wire x1="127" y1="109.22" x2="127" y2="93.98" width="0.1524" layer="91"/>
 <pinref part="IC1" gate="G$1" pin="IO3"/>
 <wire x1="127" y1="93.98" x2="134.62" y2="93.98" width="0.1524" layer="91"/>
-<wire x1="160.02" y1="111.76" x2="149.86" y2="111.76" width="0.1524" layer="91"/>
-<wire x1="149.86" y1="111.76" x2="149.86" y2="109.22" width="0.1524" layer="91"/>
 </segment>
 <segment>
@@
 </segment>
 </net>
+<net name="N$17" class="0">
+<segment>
+<pinref part="IC6" gate="G$1" pin="FORCE_AP"/>
+<pinref part="R27" gate="G$1" pin="1"/>
+<wire x1="678.18" y1="182.88" x2="673.1" y2="182.88" width="0.1524" layer="91"/>
+<wire x1="673.1" y1="182.88" x2="673.1" y2="180.34" width="0.1524" layer="91"/>
+<pinref part="TP11" gate="G$1" pin="TP"/>
+<junction x="673.1" y="182.88"/>
+</segment>
+</net>

Commit message: mostly routed
Parts:
- removed R26: TEmp, TiLDA Mk3 Parts:R-EU_0603K-SMALL
Connections:
- net N$8: no longer R26.1
Other:
- note removed: "- needed with low voltage cutoff?"
- note removed: "not sure we need this"
- note removed: "what is its idle current?"
- moved on the sheet: ANT1, C25, C26, C38, C45, IC6, J2, Q8, R17, R20, R24, R27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

Commit message: added imu
Parts:
- added C28: 0603/10u/10V/X5R, TiLDA Mk3 Parts:C-EUC0603K-SMALL
- added C30: 0603/100n/10V/X5R, TiLDA Mk3 Parts:C-EUC0603K-SMALL
- added C31: 0603/4u7/10V/X5R, TiLDA Mk3 Parts:C-EUC0603K-SMALL
- added C32: 0603/220n/10V/X5R, TiLDA Mk3 Parts:C-EUC0603K-SMALL
- added IC5: LSM9DS0, TiLDA Mk3 Parts:LSM9DS0
- added TP18, TP19, TP20: TPB1,27, TiLDA Mk3 Parts:TPB1,27
Connections:
- net TIM10_CH1 renamed I2C_SCL
- net TIM11_CH1 renamed I2C_SDA
- removed net A5: TP7.TP
- removed net LCD_ADC_X: IC3_PC.PC0, J2.X-
- removed net LCD_ADC_Y: IC3_PC.PC1, J2.Y-
- removed net LCD_X: IC3_PE.PE4, J2.X+
- removed net LCD_Y: IC3_PE.PE5, J2.Y+
- removed net N$14: LED1.C, Q3.D
- removed net N$4: C9.2, IC3_PWR.VCAP1
- removed net N$8: IC3_PC.PC13
- new net ADC_IN: IC3_PB.PB0, JP1.10
- new net FET_OUT: LED1.C, Q3.D, TP7.TP
- new net IMU_IRQ1: IC3_PC.PC2, IC5.DRDY_G
- new net IMU_IRQ2: IC3_PC.PC13, IC5.INT1_XM
- new net IMU_SCL: IC3_PC.PC0, IC5.SCL/SPC, TP19.TP
- new net IMU_SDA: IC3_PC.PC1, IC5.SDA, TP18.TP
- new net N$16: C31.2, IC5.C1_XM
- new net N$18: C32.2, IC5.SETP_XM
- new net N$19: C32.1, IC5.SETC_XM
- new net PB11: C9.2, IC3_PWR.VCAP1, JP2.10
- net +3V3: now also C28.2, C30.2, IC5.CS_G, IC5.CS_XM, IC5.VDD, IC5.VDDIO, JP1.1
- net ADC_VIN: now also IC3_PC.PC3; no longer IC3_PB.PB0
- net BOOT1: now also D1.DIN
- net CC_IRQ: now also IC3_PE.PE4; no longer IC3_PC.PC2
- net CC_RST: now also IC3_PE.PE5, TP20.TP; no longer IC3_PC.PC3
- net GND: now also C28.1, C30.1, C31.1, IC5.GND, IC5.SDO_G/SA0_G, IC5.SDO_XM/SA0_XM
- net TIM1_CH4: no longer D1.DIN
- net V_UNREG: now also JP2.1
Other:
- note added: "consider moving >"
- note added: "consider pulldowns >"
- note added: "pullup"

Commit message: zero airwires
Parts:
- added R26: 0603/120/5%, TiLDA Mk3 Parts:R-EU_0603K-SMALL
- added TP21: TPB1,27, TiLDA Mk3 Parts:TPB1,27
- JP1, JP2: value M10NOSILK -> M11PTH; device TiLDA Mk3 Parts:M10NOSILK -> SparkFun-Connectors:M11PTH
Connections:
- removed net A4: TP8.TP
- removed net N$35: LED5.A, R2.1
- removed net TIM1_CH1: JP1.6
- removed net TIM4_CH2: IC3_PD.PD13, Q8.G
- new net BUZZ: IC3_PD.PD12, R26.2
- new net N$4: R26.1, SG1.1
- new net N$8: LED5.C, R2.2
- new net TIM17_CH1: IC3_PE.PE1, Q8.G
- net +3V3: now also JP2.1, TP5.TP; no longer S3.1, S4.1, TP6.TP
- net ADC_IN: now also JP2.7; no longer JP1.10
- net CC_RST: now also IC3_PE.PE3; no longer IC3_PE.PE5
- net FET_OUT: now also TP1.TP; no longer TP7.TP
- net GND: now also JP1.11, JP2.11, S3.1, S4.1, S7.1, SG1.2, TP10.TP; no longer TP5.TP
- net I2C_SCL: now also JP2.4; no longer JP2.2
- net JOY_UP: now also IC3_PD.PD11; no longer IC3_PD.PD12
- net LCD_!RST: now also IC3_PD.PD13; no longer IC3_PE.PE1
- net N$9: now also R2.1; no longer LED5.C
- net PB11: now also JP1.7; no longer JP2.10
- net SDIO_SW: now also IC3_PA.PA8; no longer IC3_PD.PD11
- net SPI2_CLK: now also JP1.8; no longer JP2.7
- net SPI2_MISO: now also JP1.9; no longer JP2.8
- net SPI2_MOSI: now also JP1.10; no longer JP2.9
- net SPI2_NSS: now also JP1.6; no longer JP2.6
- net TEAR: now also IC3_PE.PE5, TP21.TP; no longer IC3_PE.PE3
- net TIM1_CH2: now also JP2.8; no longer JP1.7
- net TIM1_CH3: now also JP2.9; no longer JP1.8
- net TIM1_CH4: now also JP2.10; no longer JP1.9
- net TIM2_CH3: now also TP6.TP; no longer TP10.TP
- net USART6_RX: now also JP2.6, TP7.TP; no longer JP2.5, TP1.TP
- net USART6_TX: now also JP2.5; no longer JP2.4
- net VBUS: now also LED5.A; no longer R2.2
- net V_UNREG: now also JP2.2, TP8.TP; no longer JP2.1
Other:
- note added: "0 1 2 3 4 5 6 7 8 9 10 11 12 13 14 15"
- note added: "BTN MENU"
- note added: "CC_IRQ"
- note added: "EXTI List"
- note added: "IMU IRQ1"
- note added: "IMU IRQ2"
- note added: "JOY CENTRE"
- note added: "JOY_DWN"
- note added: "JOY_LEFT"
- note added: "JOY_RIGHT"
- note added: "JOY_UP"
- note added: "MOM DWN"
- note added: "MOM RIGHT"
- note added: "TEAR"
- moved on the sheet: LED5, R2, SG1

Commit message: getting there now...
Parts:
- removed C14: 0603/1u/10V/X5R, TiLDA Mk3 Parts:C-EUC0603K-SMALL
- removed R18, R19: 0603/220k/5%, TiLDA Mk3 Parts:R-EU_0603K-SMALL
- removed SJ2: SOLDERJUMPERTRACE, TiLDA Mk3 Parts:SOLDERJUMPERTRACE
Connections:
- removed net ADC_VBUS: C14.2, IC3_PC.PC4, R18.2, R19.1
- removed net AREF: L3.1, SJ2.2
- removed net USART6_RX: IC3_PC.PC7, JP2.6, TP7.TP
- removed net USART6_TX: IC3_PC.PC6, JP2.5, TP2.TP
- new net USART3_RX: IC3_PC.PC5, JP2.6, TP7.TP
- new net USART3_TX: IC3_PC.PC4, JP2.5, TP2.TP
- net +3V3: now also L3.1; no longer SJ2.1
- net CC_HIB: now also IC3_PC.PC6; no longer IC3_PC.PC5
- net GND: no longer C14.1, R19.2
- net VBUS: no longer R18.1
Other:
- note added: "SWITCH THESE!!!"
- note added: "cc_!hib"
- note removed: "WS2812 - can connect to a usart?"
- note removed: "connect i2c on pb11"
- note removed: "speaker to tim1"
- note removed: "undecided whether to bother with this"

Commit message: half way thorugh checking
Parts:
- added R18, R19: DNP (0603/10k/5%), TiLDA Mk3 Parts:R-EU_0603K-SMALL
- added R28, R29: 0603/4.7M/5%, TiLDA Mk3 Parts:R-EU_0603K-SMALL
- C1, C3: value 0603/4u7/10V/X5R -> 0603/2u2/10V/X5R
- L1: device TiLDA Mk3 Parts:INDUCTOR1210 -> TiLDA Mk3 Parts:INDUCTOR1008
- R11: value 0603/100K/5% -> DNP / 0603/100K/5%
Connections:
- net +3V3: now also R18.1, R19.1
- net GND: now also R28.2
- net I2C_SCL: now also TP7.TP
- net I2C_SDA: now also TP2.TP
- net IMU_SCL: now also R19.2
- net IMU_SDA: now also R18.2
- net N$50: now also R28.1
- net N$55: now also R29.1
- net N$57: now also R29.2
- net USART3_RX: no longer TP7.TP
- net USART3_TX: no longer TP2.TP
Other:
- note added: "4x"
- note added: "6V MAX"
- note added: "UI"
- note added: "consider switching uart for i2c"
- note added: "in theory the full 200u might not be needed"
- note added: "unclear if really needed"
- note removed: "/CC3100 UART"
- note removed: "1431303 / 2317885"
- note removed: "< should be pulled down..?"
- note removed: "BG2970 + FDS9926A;IRFML8244TRPBF"
- note removed: "DONT BOTHER - TIM1_CH1"
- note removed: "ESP8266"
- note removed: "LEDs"
- note removed: "Place Caps for 405 0R for 4x1"
- note removed: "SWITCH THESE!!!"
- note removed: "add footprint for cap"
- note removed: "buzzer, accel footprint?"
- note removed: "cc_!hib"
- note removed: "check ESP pin connections"
- note removed: "check should be the lower half >"
- note removed: "connect pin 10"
- note removed: "i2c"
- note removed: "is 3.3V fine?"
- note removed: "pullup"
- note removed: "wrong package"
- moved on the sheet: C1, C27, C28, C3, C30, C31, C32, C4, C48, C5, C6, D2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

Commit message: DONE
Parts:
- added C14: 0603/4u7/10V/X5R, TiLDA Mk3 Parts:C-EUC0603K-SMALL
- C19: value 0603/100n/10V/X5R -> 0603/100n/10V/X5R or 0 ohm
- C28: value 0603/10u/10V/X5R -> 0603/4u7/10V/X5R
- C9: value 0603/2.2u/6.3V/X5R -> 0603/2.2u/6.3V/X5R or DNP
- R21, R22: value 0603/220k/5% -> 0603/470k/5%
- R24: value 0/dnp -> 330/dnp
Connections:
- net BOOT1 renamed WS2812
- net +3V3: now also C14.2
- net GND: now also C14.1
Other:
- note added: "check this for L4"
Changed lines of the file:
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@@
 <part name="+3V5" library="supply1" deviceset="+3V3" device=""/>
 <part name="C39" library="TiLDA Mk3 Parts" deviceset="C-EU" device="C0603K-SMALL" value="0603/100n/10V/X5R"/>
-<part name="C19" library="TiLDA Mk3 Parts" deviceset="C-EU" device="C0603K-SMALL" value="0603/100n/10V/X5R"/>
+<part name="C19" library="TiLDA Mk3 Parts" deviceset="C-EU" device="C0603K-SMALL" value="0603/100n/10V/X5R or 0 ohm"/>
 <part name="C11" library="TiLDA Mk3 Parts" deviceset="C-EU" device="C0603K-SMALL" value="0603/100n/10V/X5R"/>
 <part name="C12" library="TiLDA Mk3 Parts" deviceset="C-EU" device="C0603K-SMALL" value="0603/100n/10V/X5R"/>
-<part name="C9" library="TiLDA Mk3 Parts" deviceset="C-EU" device="C0603K-SMALL" value="0603/2.2u/6.3V/X5R"/>
+<part name="C9" library="TiLDA Mk3 Parts" deviceset="C-EU" device="C0603K-SMALL" value="0603/2.2u/6.3V/X5R or DNP"/>
 <part name="GND47" library="TiLDA Mk3 Parts" deviceset="GND" device=""/>
 <part name="C16" library="TiLDA Mk3 Parts" deviceset="C-EU" device="C0603K-SMALL" value="0603/100n/10V/X5R"/>
 <part name="C15" library="TiLDA Mk3 Parts" deviceset="C-EU" device="C0603K-SMALL" value="0603/10n/25V/X7R"/>
 <part name="GND48" library="TiLDA Mk3 Parts" deviceset="GND" device=""/>
-<part name="R22" library="TiLDA Mk3 Parts" deviceset="R-EU_" device="0603K-SMALL" value="0603/220k/5%"/>
-<part name="R21" library="TiLDA Mk3 Parts" deviceset="R-EU_" device="0603K-SMALL" value="0603/220k/5%"/>
+<part name="R22" library="TiLDA Mk3 Parts" deviceset="R-EU_" device="0603K-SMALL" value="0603/470k/5%"/>
+<part name="R21" library="TiLDA Mk3 Parts" deviceset="R-EU_" device="0603K-SMALL" value="0603/470k/5%"/>
 <part name="C33" library="TiLDA Mk3 Parts" deviceset="C-EU" device="C0603K-SMALL" value="0603/1u/10V/X5R"/>
 <part name="GND49" library="TiLDA Mk3 Parts" deviceset="GND" device=""/>
@@
 <part name="R13" library="TiLDA Mk3 Parts" deviceset="R-EU_" device="0603K-SMALL" value="0603/??/5%"/>
 <part name="GND14" library="TiLDA Mk3 Parts" deviceset="GND" device=""/>
-<part name="R24" library="TiLDA Mk3 Parts" deviceset="R-EU_" device="0603K-SMALL" value="0/dnp"/>
+<part name="R24" library="TiLDA Mk3 Parts" deviceset="R-EU_" device="0603K-SMALL" value="330/dnp"/>
 <part name="U1" library="TiLDA Mk3 Parts" deviceset="USD-SOCKET-SDIO" device="DM3AT_0011"/>
 <part name="SG1" library="TiLDA Mk3 Parts" deviceset="BUZZER" device="-PKLCS1212E"/>
@@
 <part name="+3V15" library="supply1" deviceset="+3V3" device=""/>
 <part name="GND1" library="TiLDA Mk3 Parts" deviceset="GND" device=""/>
-<part name="C28" library="TiLDA Mk3 Parts" deviceset="C-EU" device="C0603K-SMALL" value="0603/10u/10V/X5R"/>
+<part name="C28" library="TiLDA Mk3 Parts" deviceset="C-EU" device="C0603K-SMALL" value="0603/4u7/10V/X5R"/>
 <part name="C30" library="TiLDA Mk3 Parts" deviceset="C-EU" device="C0603K-SMALL" value="0603/100n/10V/X5R"/>
 <part name="C31" library="TiLDA Mk3 Parts" deviceset="C-EU" device="C0603K-SMALL" value="0603/4u7/10V/X5R"/>
@@
 <part name="R28" library="TiLDA Mk3 Parts" deviceset="R-EU_" device="0603K-SMALL" value="0603/4.7M/5%"/>
 <part name="R29" library="TiLDA Mk3 Parts" deviceset="R-EU_" device="0603K-SMALL" value="0603/4.7M/5%"/>
+<part name="C14" library="TiLDA Mk3 Parts" deviceset="C-EU" device="C0603K-SMALL" value="0603/4u7/10V/X5R"/>
 </parts>
 <sheets>
@@
 <wire x1="642.62" y1="15.24" x2="645.16" y2="12.7" width="0.1524" layer="97"/>
 <wire x1="645.16" y1="12.7" x2="645.16" y2="-10.16" width="0.1524" layer="97"/>
+<text x="88.9" y="210.82" size="1.778" layer="97">check this for L4</text>
 </plain>
 <instances>
@@
 <instance part="C4" gate="G$1" x="528.32" y="121.92"/>
 <instance part="GND102" gate="1" x="528.32" y="114.3"/>
-<instance part="+3V23" gate="G$1" x="132.08" y="182.88" rot="R180"/>
+<instance part="+3V23" gate="G$1" x="129.54" y="195.58" rot="R90"/>
 <instance part="LED1" gate="G$1" x="347.98" y="162.56"/>
 <instance part="R1" gate="G$1" x="347.98" y="170.18" rot="R90"/>
@@
 <attribute name="NAME" x="641.5786" y="19.05" size="1.778" layer="95" rot="R270"/>
 <attribute name="VALUE" x="636.778" y="19.05" size="1.778" layer="96" rot="R270"/>
+</instance>
+<instance part="C14" gate="G$1" x="269.24" y="127" smashed="yes" rot="R180">
+<attribute name="NAME" x="269.621" y="127" size="1.778" layer="95" rot="R270"/>
+<attribute name="VALUE" x="271.399" y="129.54" size="1.778" layer="96" rot="R90"/>
 </instance>
 </instances>
@@
 <wire x1="279.4" y1="124.46" x2="279.4" y2="127" width="0.1524" layer="91"/>
 <junction x="274.32" y="124.46"/>
+<pinref part="C14" gate="G$1" pin="1"/>
 </segment>
 <segment>
@@
 <wire x1="274.32" y1="134.62" x2="279.4" y2="134.62" width="0.1524" layer="91"/>
 <junction x="274.32" y="134.62"/>
+<pinref part="C14" gate="G$1" pin="2"/>
+<junction x="269.24" y="132.08"/>
 </segment>
 <segment>
@@
 <pinref part="L3" gate="G$1" pin="1"/>
 <wire x1="134.62" y1="195.58" x2="132.08" y2="195.58" width="0.1524" layer="91"/>
-<label x="127" y="195.58" size="1.778" layer="95"/>
 <pinref part="+3V23" gate="G$1" pin="+3V3"/>
-<wire x1="132.08" y1="195.58" x2="127" y2="195.58" width="0.1524" layer="91"/>
-<wire x1="132.08" y1="185.42" x2="132.08" y2="195.58" width="0.1524" layer="91"/>
-<junction x="132.08" y="195.58"/>
 </segment>
 <segment>
@@
 </segment>
 </net>
-<net name="BOOT1" class="0">
+<net name="WS2812" class="0">
 <segment>
 <pinref part="IC3" gate="_PB" pin="PB2"/>
