File: cc3100-breakout.sch (EAGLE design)
At the start: 56 parts, among them IC4 CC3100, IC5 S25FL216K0PMFI011, X4 DNP - ABS07-32.768KHZ-T, X5 Q24FA20H00396, X6 MC-921

Commit message: started to rework pin mapping a little so the lcd uses the FSMC pins
Parts:
- added R4: 150, passives-7351:RESISTOR0603-N
- added TP1, TP2, TP3, TP4: TPPAD1-11, TiLDA Mk3 Parts:TPPAD1-11
Connections:
- new net N$14: LED1.C, R4.P$2
- net +3V3: now also LED1.A
- net GND: now also R4.P$1, TP4.TP
- net N$17: now also TP2.TP
- net N$18: now also TP1.TP
- net N$22: now also TP3.TP
Changed lines of the file:
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@@
 <part name="LED4" library="led" deviceset="LED" device="CHIPLED_0603"/>
 <part name="LED5" library="led" deviceset="LED" device="CHIPLED_0603"/>
+<part name="+3V2" library="supply1" deviceset="+3V3" device=""/>
+<part name="R4" library="passives-7351" deviceset="RESISTOR" device="0603-N" value="150"/>
+<part name="GND3" library="TiLDA Mk3 Parts" deviceset="GND" device=""/>
+<part name="TP1" library="TiLDA Mk3 Parts" deviceset="TP" device="PAD1-11"/>
+<part name="TP2" library="TiLDA Mk3 Parts" deviceset="TP" device="PAD1-11"/>
+<part name="TP3" library="TiLDA Mk3 Parts" deviceset="TP" device="PAD1-11"/>
+<part name="TP4" library="TiLDA Mk3 Parts" deviceset="TP" device="PAD1-11"/>
 </parts>
 <sheets>
@@
 <instance part="LED4" gate="G$1" x="246.38" y="134.62"/>
 <instance part="LED5" gate="G$1" x="259.08" y="134.62"/>
+<instance part="+3V2" gate="G$1" x="220.98" y="139.7"/>
+<instance part="R4" gate="G$1" x="220.98" y="124.46" rot="R90"/>
+<instance part="GND3" gate="1" x="220.98" y="116.84"/>
+<instance part="TP1" gate="G$1" x="10.16" y="233.68" rot="R90"/>
+<instance part="TP2" gate="G$1" x="43.18" y="213.36"/>
+<instance part="TP3" gate="G$1" x="66.04" y="193.04" rot="R90"/>
+<instance part="TP4" gate="G$1" x="10.16" y="193.04" rot="R90"/>
 </instances>
 <busses>
@@
 <pinref part="GND28" gate="1" pin="GND"/>
 <wire x1="12.7" y1="218.44" x2="12.7" y2="193.04" width="0.1524" layer="91"/>
+<pinref part="TP4" gate="G$1" pin="TP"/>
+<junction x="12.7" y="193.04"/>
 </segment>
 <segment>
@@
 <pinref part="RN1" gate="C" pin="1"/>
 <pinref part="GND2" gate="1" pin="GND"/>
+</segment>
+<segment>
+<pinref part="R4" gate="G$1" pin="P$1"/>
+<pinref part="GND3" gate="1" pin="GND"/>
 </segment>
 </net>
@@
 <pinref part="IC4" gate="_POWER" pin="LDO_IN2"/>
 <pinref part="IC4" gate="_POWER" pin="LDO_IN1"/>
+<pinref part="TP1" gate="G$1" pin="TP"/>
 </segment>
 </net>
@@
 <net name="N$17" class="0">
 <segment>
-<wire x1="43.18" y1="208.28" x2="43.18" y2="210.82" width="0.1524" layer="91"/>
 <wire x1="43.18" y1="210.82" x2="50.8" y2="210.82" width="0.1524" layer="91"/>
 <wire x1="50.8" y1="210.82" x2="55.88" y2="210.82" width="0.1524" layer="91"/>
@@
 <pinref part="C27" gate="G$1" pin="2"/>
 <pinref part="C40" gate="G$1" pin="2"/>
+<pinref part="TP2" gate="G$1" pin="TP"/>
+<junction x="43.18" y="210.82"/>
 </segment>
 </net>
@@
 <pinref part="IC4" gate="_POWER" pin="VDD_DIG1"/>
 <pinref part="IC4" gate="_POWER" pin="VDD_DIG2"/>
+<pinref part="TP3" gate="G$1" pin="TP"/>
 </segment>
 </net>
@@
 <pinref part="+3V1" gate="G$1" pin="+3V3"/>
 </segment>
+<segment>
+<pinref part="LED1" gate="G$1" pin="A"/>
+<pinref part="+3V2" gate="G$1" pin="+3V3"/>
+</segment>
 </net>
 <net name="N$5" class="0">
@@
 </segment>
 </net>
+<net name="N$14" class="0">
+<segment>
+<pinref part="LED1" gate="G$1" pin="C"/>
+<pinref part="R4" gate="G$1" pin="P$2"/>
+</segment>
+</net>
