File: Mk3 Prototype3.sch (EAGLE design)
At the start: 151 parts, among them IC1 TPD3E001DRL, IC2 TPS62082, IC3 STM32F401V, IC4 BQ24092, IC6 CC3100MOD, IC7 BQ2970, IC8 LSM6DS3, IC9 LIS3MDL, J1 ZX62-AB-5PA(11), J2 ER-CON50HT-1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

Commit message: copying switch between libs
Parts:
- S3, S4: device Mine:SWITCH-MOMENTARY-2 -> TiLDA Mk3 Parts:SWITCH-MOMENTARY-2
Changed lines of the file:
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@@
 <?xml version="1.0" encoding="utf-8"?>
 <!DOCTYPE eagle SYSTEM "eagle.dtd">
-<eagle version="6.6.0">
+<eagle version="6.5.0">
 <drawing>
 <settings>
@@
 <attribute name="FARNELL" value="1316987"/>
 </part>
-<part name="S4" library="Mine" deviceset="SWITCH-MOMENTARY-2" device="" value="1217769">
+<part name="S4" library="TiLDA Mk3 Parts" deviceset="SWITCH-MOMENTARY-2" device="" value="1217769">
 <attribute name="FARNELL" value="1217769"/>
 </part>
-<part name="S3" library="Mine" deviceset="SWITCH-MOMENTARY-2" device="" value="1217769">
+<part name="S3" library="TiLDA Mk3 Parts" deviceset="SWITCH-MOMENTARY-2" device="" value="1217769">
 <attribute name="FARNELL" value="1217769"/>
 </part>

Commit message: cc spi clk moved to allow dac, led fet moved, ws2812 on timer
Connections:
- removed net TIM1_CH3: IC3_PE.PE13, JP2.9
- new net BOOT1: IC3_PB.PB2, R11.2
- new net DAC_OUT: IC3_PA.PA5, JP2.5
- new net N$14: J2.X+
- new net N$16: J2.Y-
- new net N$18: J2.X-
- new net N$19: J2.Y+
- net ADC_IN: now also JP2.8; no longer JP2.7
- net SPI1_SCK: now also IC3_PE.PE13; no longer IC3_PA.PA5
- net TIM1_CH1N: now also IC3_PC.PC7; no longer IC3_PB.PB13
- net TIM1_CH2: now also JP2.9; no longer JP2.8
- net USART3_RX: now also JP2.7; no longer JP2.6
- net USART3_TX: now also JP2.6; no longer JP2.5
- net WS2812: now also IC3_PB.PB13; no longer IC3_PB.PB2, R11.2
Other:
- note added: "1 2 3 4 5 6 7 8 15 16 17"
- note added: "CH1-4: servos"
- note added: "CH1: Backlight"
- note added: "CH1: buzzer"
- note added: "CH1N: WS2812"
- note added: "CH2,4: headers"
- note added: "CH2: FET LED"
- note added: "Timers List"
- note added: "internal use"
- note removed: "/ BOOT1"
- moved on the sheet: R26, SG1
Changed lines of the file:
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@@
 <text x="797.56" y="104.14" size="2.54" layer="90">see if a resistor is needed on the stm32 crytal</text>
 <text x="162.56" y="17.78" size="1.778" layer="91" rot="R90">depends on led</text>
-<text x="86.36" y="198.12" size="1.778" layer="91">/ BOOT1</text>
 <text x="358.14" y="127" size="1.778" layer="91">/ JOY_CEN</text>
 <text x="129.286" y="199.136" size="1.778" layer="91" rot="R90">low ESR</text>
@@
 <text x="109.22" y="139.7" size="3.81" layer="97" ratio="15">USB OTG</text>
 <text x="500.38" y="142.24" size="3.81" layer="97" ratio="15">Power</text>
-<text x="335.28" y="203.2" size="3.81" layer="97" ratio="15">UI</text>
+<text x="281.94" y="175.26" size="3.81" layer="97" ratio="15">UI</text>
 <text x="119.38" y="66.04" size="3.81" layer="97" ratio="15">ADC Inputs</text>
 <text x="693.42" y="223.52" size="1.778" layer="91">0: parallel; 1: serial</text>
@@
 <text x="363.22" y="106.68" size="1.778" layer="91">mom_right</text>
 <text x="365.76" y="101.6" size="1.778" layer="91">mom_menu</text>
+<text x="314.96" y="246.38" size="3.81" layer="97" ratio="15">Timers List</text>
+<text x="317.5" y="203.2" size="1.6764" layer="91" ratio="11" align="bottom-right">1
+2
+3
+4
+5
+6
+7
+8
+15
+16
+17</text>
+<text x="322.58" y="223.52" size="1.778" layer="91">internal use</text>
+<wire x1="312.42" y1="231.14" x2="342.9" y2="231.14" width="0.1524" layer="97"/>
+<wire x1="320.04" y1="233.68" x2="320.04" y2="200.66" width="0.1524" layer="97"/>
+<wire x1="312.42" y1="200.66" x2="320.04" y2="200.66" width="0.1524" layer="97"/>
+<wire x1="320.04" y1="200.66" x2="342.9" y2="200.66" width="0.1524" layer="97"/>
+<text x="322.58" y="203.2" size="1.778" layer="91">CH1: Backlight</text>
+<text x="322.58" y="208.28" size="1.778" layer="91">CH1N: WS2812</text>
+<text x="322.58" y="210.82" size="1.778" layer="91">CH2: FET LED</text>
+<text x="322.58" y="226.06" size="1.778" layer="91">CH1-4: servos</text>
+<text x="322.58" y="228.6" size="1.778" layer="91">CH2,4: headers</text>
+<text x="322.58" y="220.98" size="1.778" layer="91">CH1: buzzer</text>
 </plain>
 <instances>
@@
 <attribute name="FARNELL" x="441.96" y="30.48" size="1.778" layer="96" display="off"/>
 </instance>
-<instance part="SG1" gate="G$1" x="358.14" y="190.5" smashed="yes" rot="R270">
-<attribute name="NAME" x="363.22" y="193.04" size="1.778" layer="95" rot="R270"/>
+<instance part="SG1" gate="G$1" x="304.8" y="162.56" smashed="yes" rot="R270">
+<attribute name="NAME" x="309.88" y="165.1" size="1.778" layer="95" rot="R270"/>
 </instance>
 <instance part="R27" gate="G$1" x="431.8" y="177.8" rot="R270"/>
@@
 </instance>
 <instance part="GND19" gate="1" x="330.2" y="101.6"/>
-<instance part="R26" gate="G$1" x="350.52" y="190.5" rot="R180"/>
-<instance part="GND20" gate="1" x="355.6" y="185.42"/>
+<instance part="R26" gate="G$1" x="297.18" y="162.56" rot="R180"/>
+<instance part="GND20" gate="1" x="302.26" y="157.48"/>
 <instance part="TP21" gate="G$1" x="744.22" y="132.08" smashed="yes" rot="R180">
 <attribute name="NAME" x="745.49" y="130.81" size="1.778" layer="95" rot="R180"/>
@@
 <net name="TIM1_CH1N" class="0">
 <segment>
-<pinref part="IC3" gate="_PB" pin="PB13"/>
-<wire x1="68.58" y1="167.64" x2="71.12" y2="167.64" width="0.1524" layer="91"/>
-<label x="71.12" y="167.64" size="1.778" layer="95"/>
-</segment>
-<segment>
 <wire x1="370.84" y1="149.86" x2="353.06" y2="149.86" width="0.1524" layer="91"/>
 <label x="363.22" y="149.86" size="1.778" layer="95"/>
 <pinref part="Q3" gate="G$1" pin="G"/>
 </segment>
+<segment>
+<pinref part="IC3" gate="_PC" pin="PC7"/>
+<wire x1="33.02" y1="116.84" x2="35.56" y2="116.84" width="0.1524" layer="91"/>
+<label x="35.56" y="116.84" size="1.778" layer="95"/>
+</segment>
 </net>
 <net name="N$21" class="0">
@@
 </segment>
 <segment>
-<wire x1="363.22" y1="38.1" x2="358.14" y2="38.1" width="0.1524" layer="91"/>
-<label x="358.14" y="38.1" size="1.778" layer="95" rot="MR0"/>
-<pinref part="JP2" gate="G$1" pin="8"/>
-</segment>
-</net>
-<net name="TIM1_CH3" class="0">
-<segment>
-<pinref part="IC3" gate="_PE" pin="PE13"/>
-<wire x1="73.66" y1="35.56" x2="78.74" y2="35.56" width="0.1524" layer="91"/>
-<label x="76.2" y="35.56" size="1.778" layer="95"/>
-</segment>
-<segment>
 <wire x1="358.14" y1="35.56" x2="363.22" y2="35.56" width="0.1524" layer="91"/>
 <label x="358.14" y="35.56" size="1.778" layer="95" rot="MR0"/>
@@
 <net name="SPI1_SCK" class="0">
 <segment>
-<pinref part="IC3" gate="_PA" pin="PA5"/>
-<wire x1="30.48" y1="190.5" x2="33.02" y2="190.5" width="0.1524" layer="91"/>
-<label x="33.02" y="190.5" size="1.778" layer="95"/>
-</segment>
-<segment>
 <wire x1="533.4" y1="213.36" x2="490.22" y2="213.36" width="0.1524" layer="91"/>
 <label x="525.78" y="213.36" size="1.778" layer="95"/>
 <pinref part="IC6" gate="G$1" pin="SPI_CLK"/>
 </segment>
+<segment>
+<pinref part="IC3" gate="_PE" pin="PE13"/>
+<wire x1="73.66" y1="35.56" x2="78.74" y2="35.56" width="0.1524" layer="91"/>
+<label x="76.2" y="35.56" size="1.778" layer="95"/>
+</segment>
 </net>
 <net name="SPI1_NSS" class="0">
@@
 <net name="WS2812" class="0">
 <segment>
-<pinref part="IC3" gate="_PB" pin="PB2"/>
-<label x="71.12" y="198.12" size="1.778" layer="95"/>
-<pinref part="R11" gate="G$1" pin="2"/>
-<wire x1="68.58" y1="198.12" x2="88.9" y2="198.12" width="0.1524" layer="91"/>
-<junction x="88.9" y="198.12"/>
-<wire x1="88.9" y1="198.12" x2="93.98" y2="198.12" width="0.1524" layer="91"/>
-</segment>
-<segment>
 <label x="480.06" y="106.68" size="1.778" layer="95"/>
 <pinref part="D1" gate="G$1" pin="DIN"/>
 <wire x1="485.14" y1="106.68" x2="480.06" y2="106.68" width="0.1524" layer="91"/>
 </segment>
+<segment>
+<pinref part="IC3" gate="_PB" pin="PB13"/>
+<wire x1="68.58" y1="167.64" x2="71.12" y2="167.64" width="0.1524" layer="91"/>
+<label x="71.12" y="167.64" size="1.778" layer="95"/>
+</segment>
 </net>
 <net name="N$39" class="0">
@@
 </segment>
 <segment>
-<wire x1="363.22" y1="40.64" x2="358.14" y2="40.64" width="0.1524" layer="91"/>
-<label x="358.14" y="40.64" size="1.778" layer="95" rot="MR0"/>
-<pinref part="JP2" gate="G$1" pin="7"/>
+<wire x1="363.22" y1="38.1" x2="358.14" y2="38.1" width="0.1524" layer="91"/>
+<label x="358.14" y="38.1" size="1.778" layer="95" rot="MR0"/>
+<pinref part="JP2" gate="G$1" pin="8"/>
 </segment>
 </net>
@@
 <segment>
 <pinref part="R26" gate="G$1" pin="2"/>
-<wire x1="345.44" y1="190.5" x2="327.66" y2="190.5" width="0.1524" layer="91"/>
-<label x="327.66" y="190.5" size="1.778" layer="95"/>
+<wire x1="292.1" y1="162.56" x2="274.32" y2="162.56" width="0.1524" layer="91"/>
+<label x="274.32" y="162.56" size="1.778" layer="95"/>
 </segment>
 </net>
@@
 </segment>
 <segment>
-<wire x1="363.22" y1="45.72" x2="358.14" y2="45.72" width="0.1524" layer="91"/>
-<label x="358.14" y="45.72" size="1.778" layer="95" rot="MR0"/>
-<pinref part="JP2" gate="G$1" pin="5"/>
+<wire x1="363.22" y1="43.18" x2="358.14" y2="43.18" width="0.1524" layer="91"/>
+<label x="358.14" y="43.18" size="1.778" layer="95" rot="MR0"/>
+<pinref part="JP2" gate="G$1" pin="6"/>
 </segment>
 </net>
@@
 </segment>
 <segment>
-<wire x1="363.22" y1="43.18" x2="358.14" y2="43.18" width="0.1524" layer="91"/>
-<label x="358.14" y="43.18" size="1.778" layer="95" rot="MR0"/>
-<pinref part="JP2" gate="G$1" pin="6"/>
+<wire x1="363.22" y1="40.64" x2="358.14" y2="40.64" width="0.1524" layer="91"/>
+<label x="358.14" y="40.64" size="1.778" layer="95" rot="MR0"/>
+<pinref part="JP2" gate="G$1" pin="7"/>
 </segment>
 </net>
@@
 </segment>
 </net>
+<net name="DAC_OUT" class="0">
+<segment>
+<pinref part="IC3" gate="_PA" pin="PA5"/>
+<wire x1="30.48" y1="190.5" x2="33.02" y2="190.5" width="0.1524" layer="91"/>
+<label x="33.02" y="190.5" size="1.778" layer="95"/>
+</segment>
+<segment>
+<wire x1="363.22" y1="45.72" x2="358.14" y2="45.72" width="0.1524" layer="91"/>
+<label x="358.14" y="45.72" size="1.778" layer="95" rot="MR0"/>
+<pinref part="JP2" gate="G$1" pin="5"/>
+</segment>
+</net>
+<net name="BOOT1" class="0">
+<segment>
+<pinref part="IC3" gate="_PB" pin="PB2"/>
+<label x="71.12" y="198.12" size="1.778" layer="95"/>
+<pinref part="R11" gate="G$1" pin="2"/>
+<wire x1="68.58" y1="198.12" x2="88.9" y2="198.12" width="0.1524" layer="91"/>
+<junction x="88.9" y="198.12"/>
+<wire x1="88.9" y1="198.12" x2="93.98" y2="198.12" width="0.1524" layer="91"/>
+</segment>
+</net>
+<net name="N$14" class="0">
+<segment>
+<pinref part="J2" gate="G$1" pin="X+"/>
+<wire x1="754.38" y1="119.38" x2="751.84" y2="119.38" width="0.1524" layer="91"/>
+</segment>
+</net>
+<net name="N$16" class="0">
+<segment>
+<pinref part="J2" gate="G$1" pin="Y-"/>
+<wire x1="751.84" y1="111.76" x2="754.38" y2="111.76" width="0.1524" layer="91"/>
+</segment>
+</net>
+<net name="N$18" class="0">
+<segment>
+<pinref part="J2" gate="G$1" pin="X-"/>
+<wire x1="754.38" y1="116.84" x2="751.84" y2="116.84" width="0.1524" layer="91"/>
+</segment>
+</net>
+<net name="N$19" class="0">
+<segment>
+<pinref part="J2" gate="G$1" pin="Y+"/>
+<wire x1="754.38" y1="114.3" x2="751.84" y2="114.3" width="0.1524" layer="91"/>
+</segment>
+</net>

Commit message: sch mostly done for 0.3
Parts:
- removed C20, C21: DNP (0603/10p/50V/NP0), TiLDA Mk3 Parts:C-EUC0603K-SMALL
- removed R43: DNP (0603/150/5%), TiLDA Mk3 Parts:R-EU_0603K-SMALL
- removed X2: DNP (16MHz-3.2-2.5), TiLDA Mk3 Parts:CRYSTAL-3.2-2.5
- added S1: SWITCH-MOMENTARY-2SMD-1101NE, SparkFun-Electromechanical:SWITCH-MOMENTARY-2SMD-1101NE
- added SJ2: JUMPER-PAD-3-2OF3_NC_BY_TRACE_SMALL, SparkFun-Passives:JUMPER-PAD-3-2OF3_NC_BY_TRACE_SMALL
- added TP2, TP3: TPB1,27, TiLDA Mk3 Parts:TPB1,27
Connections:
- removed net IMU_IRQ1: IC3_PC.PC2, TP1.TP
- removed net N$14: J2.X+
- removed net N$15: D3.C, Q1.E2, Q2.S, Q6.S, R45.1
- removed net N$18: J2.X-
- removed net N$19: J2.Y+
- removed net N$31: C21.2, IC3_PH.PH0/OCS_IN, X2.C2
- removed net N$33: C20.2, R43.2, X2.C1
- removed net N$42: IC3_PH.PH1/OSC_OUT, R43.1
- new net ADC_X: IC3_PC.PC2, J2.X-
- new net ADC_Y: IC3_PC.PC3, J2.Y-
- new net T_X: IC3_PH.PH0/OCS_IN, J2.X+
- new net T_Y: IC3_PH.PH1/OSC_OUT, J2.Y+
- net +3V3: now also SJ2.1
- net ADC_VIN: now also IC3_PA.PA1; no longer IC3_PC.PC3
- net GND: now also S1.2, SJ2.3; no longer C20.1, C21.1, X2.GND@1, X2.GND@2
- net LCD0: now also TP1.TP
- net LCD_MODE: now also SJ2.2
- net LCD_RD: now also TP2.TP
- net LCD_WRX: now also TP3.TP
- net N$16: now also D2.A, Q1.E1, Q2.D, Q6.D; no longer J2.Y-
- net NRST: now also S1.1
- net SPI3_SCK: now also JP1.3, OUTLINE1.CH3
- net TIM2_CH2: no longer IC3_PA.PA1, JP1.3, OUTLINE1.CH3
- net VBAT: now also Q6.S, R45.1; no longer Q1.E1, Q2.D
- net V_UNREG: now also D3.C, Q1.E2, Q2.S; no longer D2.A, Q6.D
Other:
- moved on the sheet: D2, D3, Q1, Q2, Q6, R15, R16, R45, S5, SJ1, TP1

Commit message: rearranged gpio, one gpio is now NC...
Connections:
- net ADC_VIN: now also IC3_PA.PA3; no longer IC3_PA.PA1
- net PB11: no longer C9.2, IC3_PWR.VCAP1
- net SPI3_SCK: no longer JP1.3, OUTLINE1.CH3
- net TIM2_CH2: now also IC3_PA.PA1, JP1.3, OUTLINE1.CH3
- net TIM2_CH4: now also C9.2, IC3_PWR.VCAP1; no longer IC3_PA.PA3
Changed lines of the file:
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@@
 <net name="PB11" class="0">
-<segment>
-<pinref part="C9" gate="G$1" pin="2"/>
-<pinref part="IC3" gate="_PWR" pin="VCAP1"/>
-<wire x1="165.1" y1="205.74" x2="162.56" y2="205.74" width="0.1524" layer="91"/>
-<wire x1="165.1" y1="205.74" x2="165.1" y2="208.28" width="0.1524" layer="91"/>
-<wire x1="165.1" y1="208.28" x2="175.26" y2="208.28" width="0.1524" layer="91"/>
-<label x="172.72" y="208.28" size="1.778" layer="95"/>
-<junction x="165.1" y="205.74"/>
-</segment>
 <segment>
 <wire x1="332.74" y1="40.64" x2="327.66" y2="40.64" width="0.1524" layer="91"/>
@@
 <pinref part="R24" gate="G$1" pin="1"/>
 </segment>
-<segment>
-<wire x1="332.74" y1="50.8" x2="325.12" y2="50.8" width="0.1524" layer="91"/>
-<label x="327.66" y="50.8" size="1.778" layer="95" rot="MR0"/>
-<pinref part="JP1" gate="G$1" pin="3"/>
-</segment>
-<segment>
-<wire x1="543.56" y1="43.18" x2="543.56" y2="45.72" width="0.1524" layer="91"/>
-<label x="543.56" y="45.72" size="1.778" layer="95" rot="R90"/>
-<pinref part="OUTLINE1" gate="G$1" pin="CH3"/>
-</segment>
 </net>
 <net name="SPI3_MOSI" class="0">
@@
 </segment>
 <segment>
-<pinref part="IC3" gate="_PA" pin="PA1"/>
-<wire x1="30.48" y1="200.66" x2="33.02" y2="200.66" width="0.1524" layer="91"/>
-<label x="33.02" y="200.66" size="1.778" layer="95"/>
+<wire x1="33.02" y1="195.58" x2="30.48" y2="195.58" width="0.1524" layer="91"/>
+<label x="33.02" y="195.58" size="1.778" layer="95"/>
+<pinref part="IC3" gate="_PA" pin="PA3"/>
 </segment>
 </net>
@@
 <label x="431.8" y="78.74" size="1.778" layer="95"/>
 </segment>
+<segment>
+<wire x1="543.56" y1="43.18" x2="543.56" y2="45.72" width="0.1524" layer="91"/>
+<label x="543.56" y="45.72" size="1.778" layer="95" rot="R90"/>
+<pinref part="OUTLINE1" gate="G$1" pin="CH3"/>
+</segment>
+<segment>
+<wire x1="332.74" y1="50.8" x2="325.12" y2="50.8" width="0.1524" layer="91"/>
+<label x="327.66" y="50.8" size="1.778" layer="95" rot="MR0"/>
+<pinref part="JP1" gate="G$1" pin="3"/>
+</segment>
+<segment>
+<pinref part="IC3" gate="_PA" pin="PA1"/>
+<wire x1="30.48" y1="200.66" x2="33.02" y2="200.66" width="0.1524" layer="91"/>
+<label x="33.02" y="200.66" size="1.778" layer="95"/>
+</segment>
 </net>
 <net name="TIM2_CH3" class="0">
@@
 <net name="TIM2_CH4" class="0">
 <segment>
-<wire x1="33.02" y1="195.58" x2="30.48" y2="195.58" width="0.1524" layer="91"/>
-<label x="33.02" y="195.58" size="1.778" layer="95"/>
-<pinref part="IC3" gate="_PA" pin="PA3"/>
-</segment>
-<segment>
 <pinref part="SV4" gate="G$1" pin="3"/>
 <wire x1="424.18" y1="116.84" x2="434.34" y2="116.84" width="0.1524" layer="91"/>
@@
 <pinref part="OUTLINE1" gate="G$1" pin="CH1"/>
 </segment>
-</net>
+<segment>
+<pinref part="C9" gate="G$1" pin="2"/>
+<pinref part="IC3" gate="_PWR" pin="VCAP1"/>
+<wire x1="165.1" y1="205.74" x2="162.56" y2="205.74" width="0.1524" layer="91"/>
+<wire x1="165.1" y1="205.74" x2="165.1" y2="208.28" width="0.1524" layer="91"/>
+<wire x1="165.1" y1="208.28" x2="175.26" y2="208.28" width="0.1524" layer="91"/>
+<label x="172.72" y="208.28" size="1.778" layer="95"/>
+<junction x="165.1" y="205.74"/>
+</segment>
+</net>
