File: Mk3 Prototype3.sch (EAGLE design)
At the start: 150 parts, among them IC1 TPD3E001DRL, IC2 TPS62082, IC3 STM32F401V, IC4 BQ24092, IC6 CC3100MOD, IC7 BQ2970, IC8 LSM6DS3, IC9 LIS3MDL, J1 ZX62-AB-5PA(11), J2 ER-CON50HT-1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

Commit message: silk tidied
Connections:
- net TIM1_CH1N renamed TIM8_CH2
Changed lines of the file:
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@@
 </segment>
 </net>
-<net name="TIM1_CH1N" class="0">
+<net name="TIM8_CH2" class="0">
 <segment>
 <wire x1="370.84" y1="149.86" x2="353.06" y2="149.86" width="0.1524" layer="91"/>

Commit message: Rework entier power section layout on schematic
Parts:
- JP3: value (none) -> JST PH 2mm
- R32: value DNP (0) -> DNP (0603/0R/5%)
Connections:
- net N$16 renamed VABT_SWTICHED
- net N$57 renamed VBAT_NEG
Other:
- note added: "+"
- note added: "-"
- note added: "3V3 Regulator"
- note added: "Battery Charger"
- note added: "Battery Connection"
- note added: "Battery Switch"
- note added: "Battery portection bypass"
- note added: "Battery protection"
- note added: "Ideal Diode"
- note added: "LCD Screen"
- note added: "LCD_MODE 0: parallel; 1: serial"
- note added: "OTG Supply From Battery"
- note added: "Outline Conductive Pads"
- note added: "Power Supply and Charging"
- note added: "USB feed and protection"
- note added: "Usb power in"
- note added: "WiFI"
- note removed: "0: parallel; 1: serial"
- note removed: "4x"
- note removed: "GRM32ER60J107ME20L"
- note removed: "LCD Connector"
- note removed: "Power"
- note removed: "SRN2512-2R2M"
- note removed: "add small resistors to stop shorting agaoinst vcc/gnd"
- note removed: "bq24092/3"
- note removed: "consider switching uart for i2c"
- note removed: "depends on whether battery has thermistor"
- note removed: "http://processors.wiki.ti.com/index.php/CC3100_Production_Line_Guide#Programming_the_CC3100_QFN_in_the_Production_Line"
- note removed: "in theory the full 200u might not be needed"
- note removed: "or change to 1x22u"
- note removed: "unclear if really needed"
- note removed: "will probably want changing to the smaller version"
- moved on the sheet: ANT1, C1, C25, C26, C27, C3, C38, C4, C45, C48, C5, C6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

Commit message: changing 4R7 -> 12R, more schematic tidying
Parts:
- R11: value DNP / 0603/100K/5% -> DNP
- R44, R47, R48, R49: value 0603/4R7/5% -> 0603/12R/5%
Other:
- note added: "Port F"
- note added: "Power selection"
- note removed: "DNP for L4"
- note removed: "IMU IRQ1"
- note removed: "STM Main Xtal"
- note removed: "USB feed and protection"
- note removed: "check this for L4"
- note removed: "consider better switches"
- note removed: "need to jumper between Vin/Vbat"
- note removed: "values depend on crystal"
- moved on the sheet: C1, C10, C15, C16, C2, C23, C24, C27, C29, C3, C33, C4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

Commit message: Revert Prototype3 files to as sent for PCB fab
Parts:
- JP3: value JST PH 2mm -> (none)
- R11: value DNP -> DNP / 0603/100K/5%
- R32: value DNP (0603/0R/5%) -> DNP (0)
- R44, R47, R48, R49: value 0603/12R/5% -> 0603/4R7/5%
Connections:
- net VABT_SWTICHED renamed N$16
- net VBAT_NEG renamed N$57
Other:
- note added: "0: parallel; 1: serial"
- note added: "4x"
- note added: "DNP for L4"
- note added: "GRM32ER60J107ME20L"
- note added: "IMU IRQ1"
- note added: "LCD Connector"
- note added: "Power"
- note added: "SRN2512-2R2M"
- note added: "STM Main Xtal"
- note added: "add small resistors to stop shorting agaoinst vcc/gnd"
- note added: "bq24092/3"
- note added: "check this for L4"
- note added: "consider better switches"
- note added: "consider switching uart for i2c"
- note added: "depends on whether battery has thermistor"
- note added: "http://processors.wiki.ti.com/index.php/CC3100_Production_Line_Guide#Programming_the_CC3100_QFN_in_the_Production_Line"
- note added: "in theory the full 200u might not be needed"
- note added: "need to jumper between Vin/Vbat"
- note added: "or change to 1x22u"
- note added: "unclear if really needed"
- note added: "values depend on crystal"
- note added: "will probably want changing to the smaller version"
- note removed: "+"
- note removed: "-"
- note removed: "3V3 Regulator"
- note removed: "Battery Charger"
- note removed: "Battery Connection"
- note removed: "Battery Switch"
- note removed: "Battery portection bypass"
- note removed: "Battery protection"
- note removed: "Ideal Diode"
- note removed: "LCD Screen"
- note removed: "LCD_MODE 0: parallel; 1: serial"
- note removed: "OTG Supply From Battery"
- note removed: "Outline Conductive Pads"
- note removed: "Port F"
- note removed: "Power Supply and Charging"
- note removed: "Power selection"
- note removed: "Usb power in"
- note removed: "WiFI"
- moved on the sheet: ANT1, C1, C10, C15, C16, C2, C23, C24, C25, C26, C27, C29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
