File: Mk3 v3.1415926535.brd (EAGLE design)
At the start: 121.6 x 70 mm, 152 parts, among them IC1 TPD3E001DRL, IC2 TPS62082, IC3 STM32F401V, IC4 BQ24092, IC6 CC3100MOD, IC7 BQ2970, IC8 LSM6DS3, IC9 LIS3MDL, J1 ZX62-AB-5PA(11), J2 ER-CON50HT-1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

Commit message: Library updates
Parts:
- LOGO3: value MICROPYTHON-STOP -> MICROPYTHON-SILK; device TiLDA Mk3 Parts:UPYTHON_LOGO_STOPONLY -> TiLDA Mk3 Parts:UPYTHON_LOGO_SLIKONLY
- moved LOGO3 10.0 mm to (107.1, 47.3), flipped to the bottom
Changed lines of the file:
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@@
 <variant name="L4" populate="no"/>
 </element>
-<element name="LOGO3" library="TiLDA Mk3 Parts" package="UPYTHON_LOGO_STOPONLY" value="MICROPYTHON-STOP" x="97.1" y="47.3">
+<element name="LOGO3" library="TiLDA Mk3 Parts" package="UPYTHON_LOGO_SLIKONLY" value="MICROPYTHON-SILK" x="107.1" y="47.3" rot="MR0">
 <variant name="L4" populate="no"/>
 </element>
