File: Mk3 v3.1415926535.brd (EAGLE design)
At the start: 121.6 x 70 mm, 154 parts, among them IC1 TPD3E001DRL, IC2 TPS62082, IC3 STM32L475VG, IC4 BQ24092, IC6 CC3100MOD-LWK, IC7 BQ2970, IC8 LSM6DS3, IC9 LIS3MDL, J1 ZX62-AB-5PA(11), J2 ER-CON50HT-1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

Commit message: Update all values for L4 variant by default
Parts:
- ANT1: value CHIPANT -> 2450AT42A100E
- C19: value 0603/100n/10V/X5R or 0 ohm -> 0603/0R
- C29: value 0603/2.2u/6.3V/X5R -> 0603/100n/10V/X5R
- C48: value 0603/100n/10V/X5R -> DNP (0603/100n/10V/X5R)
- C9: value 0603/2.2u/6.3V/X5R or DNP -> DNP
- IC6: value CC3100MOD-LWK -> CC3100MOD
- IC7: value BQ2970 -> DNP (BQ2970)
- J3: value 2x5 1.27mm -> 2x5 1.27mm (NP)
- JP1, JP2: value M11PTH -> (NP)
- JP4: value TC2030-SWDNL -> (NP)
- L2, L3: value Bead -> BLM18KG121TN1D
- LOGO1: value OSHW-LOGOM -> OSHW-LOGOM (NP)
- LOGO2: value LOGO_TI-4MM -> LOGO_TI-4MM (NP)
- LOGO3: value LOGO_ST-4MM -> LOGO_ST-4MM (NP)
- LOGO4: value LOGO_HCD-4MM -> LOGO_HCD-4MM (NP)
- LOGO5: value LOGO_MICROSOFT-4MM -> LOGO_MICROSOFT-4MM (NP)
- LOGO6: value LOGO_MICROPYTHON-8MM -> LOGO_MICROPYTHON-8MM (NP)
- OUTLINE1: value TILDA_MK3_BOARDOUTLINE -> TILDA_MK3 (NP)
- Q4: value CSD85301Q2 -> DNP (CSD85301Q2)
- R12: value 0603/150/5% -> 0603/150R/5%
- R14, R26: value 0603/120/5% -> 0603/120R/5%
- R2: value 0603/330/5% -> 0603/1k/5%
- R28, R29: value 0603/4M7/5% -> DNP (0603/4M7/5%)
- R32: value DNP (0603/0R/5%) -> 0603/0R
- R50: value 0603/2k/5% -> DNP (0603/2k/5%)
- R51: value 0603/330/5% -> DNP (0603/330/5%)
- R7: value DNP or 0603/0R/5% -> 0603/0R
- R8: value DNP or 0 -> DNP
- S5: value Power Switch -> CUS-12TB
- SJ1: value SOLDERJUMPERNO -> OTG (NP)
- SV2, SV3, SV4, SV5, SV6, SV7: value (none) -> (NP)
- SW1: value JOYSTICK_MINI_MULTICOM_NOSILK -> JOYSTICK
- TP1, TP11, TP12, TP13, TP14, TP15, TP16, TP17, TP18, TP19, TP2, TP20, TP21, TP3, TP4, TP5: value TPB1,27 -> (NP)
- U1: value USD-SOCKET-SDIO -> USD-SOCKET
- U2: value ER-TFT024-3 -> ER-TFT024-3 (NP)
Connections:
- net CC_HIB renamed !CC_HIB
- net CC_RST renamed !CC_RST
- net N$17 renamed FORCE_AP
- net N$39 renamed !UART_CTS
- net N$41 renamed SOP2
- net N$43 renamed CC_RESERVED
- net N$44 renamed !UART_RTS
- net N$61 renamed TEST_58
- net N$65 renamed TEST_59
- net N$66 renamed TEST_60
- net N$67 renamed TEST_62

Commit message: Updating LED resistor values
Parts:
- R12: value 0603/150R/5% -> 0603/2k/5%
- R14: value 0603/120R/5% -> 0603/4k7/5%
- R2: value 0603/1k/5% -> 0603/4k7/5%
- R5: value 0603/2M2/5% -> 0603/4M7/5%
Changed lines of the file:
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@@
 <attribute name="FARNELL" value="2449874" x="21.4" y="6.1" size="1.778" layer="27" rot="R180" display="off"/>
 </element>
-<element name="R2" library="TiLDA Mk3 Parts" package="C0603K-SMALL" value="0603/1k/5%" x="4.4" y="10.2" smashed="yes" rot="MR180">
+<element name="R2" library="TiLDA Mk3 Parts" package="C0603K-SMALL" value="0603/4k7/5%" x="4.4" y="10.2" smashed="yes" rot="MR180">
 <attribute name="NAME" x="3.311" y="9.4015" size="1.016" layer="26" font="vector" ratio="14" rot="MR180"/>
 </element>
@@
 <attribute name="NAME" x="33.611" y="12.5015" size="1.016" layer="26" font="vector" ratio="14" rot="MR180"/>
 </element>
-<element name="R5" library="TiLDA Mk3 Parts" package="C0603K-SMALL" value="0603/2M2/5%" x="24.6" y="3.4" smashed="yes" rot="MR90">
+<element name="R5" library="TiLDA Mk3 Parts" package="C0603K-SMALL" value="0603/4M7/5%" x="24.6" y="3.4" smashed="yes" rot="MR90">
 <attribute name="NAME" x="23.8015" y="4.289" size="1.016" layer="26" font="vector" ratio="14" rot="MR270"/>
 </element>
@@
 <attribute name="COLOUR" value="GREEN" x="27.1" y="20.6" size="1.778" layer="27" rot="R270" display="off"/>
 </element>
-<element name="R12" library="TiLDA Mk3 Parts" package="C0603K-SMALL" value="0603/150R/5%" x="28.2" y="12.4" smashed="yes" rot="MR90">
+<element name="R12" library="TiLDA Mk3 Parts" package="C0603K-SMALL" value="0603/2k/5%" x="28.2" y="12.4" smashed="yes" rot="MR90">
 <attribute name="NAME" x="28.7015" y="10.889" size="1.016" layer="26" font="vector" ratio="14" rot="MR270"/>
 </element>
-<element name="R14" library="TiLDA Mk3 Parts" package="C0603K-SMALL" value="0603/120R/5%" x="31" y="14.2" smashed="yes" rot="MR0">
+<element name="R14" library="TiLDA Mk3 Parts" package="C0603K-SMALL" value="0603/4k7/5%" x="31" y="14.2" smashed="yes" rot="MR0">
 <attribute name="NAME" x="32.511" y="14.8015" size="1.016" layer="26" font="vector" ratio="14" rot="MR180"/>
 </element>

Commit message: Correct joystick trace names
Parts:
- R18, R19: value DNP (0603/10k/5%) -> 0603/4k7/5%
- turned U1 to 0 degrees
Connections:
- net JOY_DOWN: now also IC3.56, SW1.D; no longer IC3.57, SW1.B
- net JOY_LEFT: now also IC3.87, SW1.C; no longer IC3.56, SW1.D
- net JOY_RIGHT: now also IC3.57, SW1.B; no longer IC3.87, SW1.C
Routing:
- net JOY_RIGHT: track 143.2 -> 110.1 mm, vias 7 -> 1
- net JOY_LEFT: track 110.9 -> 143.2 mm, vias 1 -> 7
- net JOY_DOWN: track 110.1 -> 110.9 mm
Other:
- board text added: "U1"
Changed lines of the file:
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@@
 <text x="95.9000125" y="24.200003125" size="0.8128" layer="21" font="vector" ratio="15" rot="SR135">SW1</text>
 <text x="50.017425" y="29.52000625" size="1.016" layer="22" ratio="15" rot="MR0">X3</text>
+<text x="18.55" y="24.75" size="1.016" layer="22" ratio="15" rot="MR90">U1</text>
 </plain>
 <attributes>
@@
 <attribute name="NAME" x="39.05" y="60.2" size="1.016" layer="26" font="vector" ratio="14" rot="MR90"/>
 </element>
-<element name="U1" library="TiLDA Mk3 Parts" package="0011XAAX09X" value="USD-SOCKET" x="6.8" y="35.6" smashed="yes" rot="MR90">
-<attribute name="NAME" x="18.55" y="24.75" size="1.016" layer="22" font="vector" ratio="14" rot="MR90"/>
-<attribute name="FARNELL" value="2427719" x="6.8" y="35.6" size="1.778" layer="28" rot="MR90" display="off"/>
+<element name="U1" library="TiLDA Mk3 Parts" package="0011XAAX09X" value="USD-SOCKET" x="6.8" y="35.6" smashed="yes" rot="MR0">
+<attribute name="NAME" x="17.65" y="47.35" size="1.016" layer="26" font="vector" ratio="14" rot="MR0"/>
+<attribute name="FARNELL" value="2427719" x="6.8" y="35.6" size="1.778" layer="28" rot="MR0" display="off"/>
 </element>
 <element name="SG1" library="TiLDA Mk3 Parts" package="BUZZER-PKLCS1212E" value="BUZZER-PKLCS1212E" x="8.4" y="47.6" smashed="yes" rot="MR0">
@@
 <element name="JP1" library="TiLDA Mk3 Parts" package="1X11" value="(NP)" x="85.68" y="3.2" smashed="yes" rot="MR0"/>
 <element name="JP2" library="TiLDA Mk3 Parts" package="1X11" value="(NP)" x="55.2" y="3.2" smashed="yes" rot="MR0"/>
-<element name="R18" library="TiLDA Mk3 Parts" package="C0603K-SMALL" value="DNP (0603/10k/5%)" x="60.7" y="19.1" smashed="yes" rot="MR180">
+<element name="R18" library="TiLDA Mk3 Parts" package="C0603K-SMALL" value="0603/4k7/5%" x="60.7" y="19.1" smashed="yes" rot="MR180">
 <attribute name="NAME" x="59.2" y="18.45" size="1.016" layer="26" font="vector" ratio="14" rot="MR180"/>
 </element>
-<element name="R19" library="TiLDA Mk3 Parts" package="C0603K-SMALL" value="DNP (0603/10k/5%)" x="63.9" y="19.1" smashed="yes" rot="MR0">
+<element name="R19" library="TiLDA Mk3 Parts" package="C0603K-SMALL" value="0603/4k7/5%" x="63.9" y="19.1" smashed="yes" rot="MR0">
 <attribute name="NAME" x="62.5" y="18.45" size="1.016" layer="26" font="vector" ratio="14" rot="MR180"/>
 </element>
@@
 <wire x1="21.6" y1="28.20710625" x2="21.6" y2="28.6" width="0.2" layer="16"/>
 <via x="28.2" y="29.6" extent="1-16" drill="0.3"/>
-<wire x1="27.4" y1="26" x2="27.4" y2="28.59289375" width="0.2" layer="16"/>
+<wire x1="27.4" y1="25.1" x2="27.4" y2="28.59289375" width="0.2" layer="16"/>
 <wire x1="24.45" y1="26" x2="25.11715625" y2="26" width="0.2" layer="16"/>
 <wire x1="25.11715625" y1="26" x2="25.258578125" y2="25.941421875" width="0.2" layer="16" curve="-45"/>
@@
 <wire x1="26.3" y1="24.6" x2="26.9" y2="24.6" width="0.2" layer="16"/>
 <wire x1="26.9" y1="24.6" x2="27.4" y2="25.1" width="0.2" layer="16" curve="90"/>
-<wire x1="27.4" y1="25.1" x2="27.4" y2="25.98284375" width="0.2" layer="16"/>
-<wire x1="27.4" y1="25.98284375" x2="27.4" y2="26" width="0.2" layer="16"/>
 <wire x1="27.4" y1="28.59289375" x2="27.546446875" y2="28.946446875" width="0.2" layer="16" curve="-45"/>
 <wire x1="27.546446875" y1="28.946446875" x2="28.2" y2="29.6" width="0.2" layer="16"/>
@@
 <wire x1="19.7857875" y1="26" x2="20.49289375" y2="25.70710625" width="0.2" layer="1" curve="-45"/>
 </signal>
-<signal name="JOY_RIGHT">
+<signal name="JOY_LEFT">
 <contactref element="IC3" pad="87"/>
 <via x="33" y="35.8" extent="1-16" drill="0.3"/>
@@
 <wire x1="99.7" y1="27.4857875" x2="99.7" y2="26.9110875" width="0.2" layer="1"/>
 </signal>
-<signal name="JOY_LEFT">
+<signal name="JOY_DOWN">
 <contactref element="IC3" pad="56"/>
 <wire x1="85.6" y1="14.8" x2="85.4" y2="14.6" width="0.2" layer="1"/>
@@
 <wire x1="47.058578125" y1="38.058578125" x2="47.2" y2="38.4" width="0.2" layer="16" curve="45"/>
 </signal>
-<signal name="JOY_DOWN">
+<signal name="JOY_RIGHT">
 <contactref element="IC3" pad="57"/>
 <via x="86.6" y="14.3" extent="1-16" drill="0.3"/>

Commit message: Publish Final Artwork files
Parts:
- added ARTWORK1: ARTWORK_MKπ_BACK, TiLDA Mk3 Parts:TILDA_MKπ_ARTWORK_BACK
- added ARTWORK2: ARTWORK_MKπ_FRONT, TiLDA Mk3 Parts:TILDA_MKπ_ARTWORK_FRONT
- OUTLINE1: device TiLDA Mk3 Parts:TILDA_MKE_OUTLINE -> TiLDA Mk3 Parts:TILDA_MKπ_OUTLINE
Changed lines of the file:
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@@
 <setting verticaltext="up"/>
 </settings>
-<grid distance="0.1" unitdist="mm" unit="mm" style="lines" multiple="1" display="yes" altdistance="0.05" altunitdist="mm" altunit="mm"/>
+<grid distance="10" unitdist="mm" unit="mm" style="lines" multiple="1" display="yes" altdistance="5" altunitdist="mm" altunit="mm"/>
 <layers>
 <layer number="1" name="Top" color="4" fill="1" visible="yes" active="yes"/>
@@
 <layer number="29" name="tStop" color="7" fill="3" visible="yes" active="yes"/>
 <layer number="30" name="bStop" color="7" fill="6" visible="yes" active="yes"/>
-<layer number="31" name="tCream" color="7" fill="4" visible="yes" active="yes"/>
-<layer number="32" name="bCream" color="7" fill="5" visible="yes" active="yes"/>
+<layer number="31" name="tCream" color="7" fill="4" visible="no" active="yes"/>
+<layer number="32" name="bCream" color="7" fill="5" visible="no" active="yes"/>
 <layer number="33" name="tFinish" color="6" fill="3" visible="no" active="yes"/>
 <layer number="34" name="bFinish" color="6" fill="6" visible="no" active="yes"/>
@@
 <layer number="37" name="tTest" color="7" fill="1" visible="no" active="yes"/>
 <layer number="38" name="bTest" color="7" fill="1" visible="no" active="yes"/>
-<layer number="39" name="tKeepout" color="4" fill="11" visible="yes" active="yes"/>
-<layer number="40" name="bKeepout" color="1" fill="11" visible="yes" active="yes"/>
-<layer number="41" name="tRestrict" color="4" fill="10" visible="yes" active="yes"/>
-<layer number="42" name="bRestrict" color="1" fill="10" visible="yes" active="yes"/>
-<layer number="43" name="vRestrict" color="2" fill="10" visible="yes" active="yes"/>
+<layer number="39" name="tKeepout" color="4" fill="11" visible="no" active="yes"/>
+<layer number="40" name="bKeepout" color="1" fill="11" visible="no" active="yes"/>
+<layer number="41" name="tRestrict" color="4" fill="10" visible="no" active="yes"/>
+<layer number="42" name="bRestrict" color="1" fill="10" visible="no" active="yes"/>
+<layer number="43" name="vRestrict" color="2" fill="10" visible="no" active="yes"/>
 <layer number="44" name="Drills" color="7" fill="1" visible="no" active="yes"/>
 <layer number="45" name="Holes" color="7" fill="1" visible="no" active="yes"/>
@@
 <attribute name="NAME" x="59.25" y="22.8" size="1.016" layer="26" ratio="14" rot="MR90"/>
 </element>
-<element name="OUTLINE1" library="TiLDA Mk3 Parts" package="TILDA_MKE_OUTLINE" value="TILDA_MK3 (NP)" x="0" y="0"/>
+<element name="OUTLINE1" library="TiLDA Mk3 Parts" package="TILDA_MKπ_OUTLINE" value="TILDA_MK3 (NP)" x="0" y="0"/>
 <element name="U2" library="TiLDA Mk3 Parts" package="ER-TFT024-3" value="ER-TFT024-3 (NP)" x="89.2" y="19.6" rot="R90"/>
 <element name="R32" library="TiLDA Mk3 Parts" package="C0603K-SMALL" value="0603/0R" x="49.6" y="52.2" smashed="yes" rot="MR90">
@@
 <element name="LOGO4" library="TiLDA Mk3 Parts" package="LOGO_HDC_4MM" value="LOGO_HCD-4MM (NP)" x="99" y="41" rot="MR0"/>
 <element name="LOGO6" library="TiLDA Mk3 Parts" package="LOGO_MICROPYTHON_8MM" value="LOGO_MICROPYTHON-8MM (NP)" x="105" y="47" rot="MR0"/>
+<element name="ARTWORK1" library="TiLDA Mk3 Parts" package="TILDA_MKπ_ARTWORK_BACK" value="ARTWORK_MKπ_BACK" x="0" y="0" rot="MR0"/>
+<element name="ARTWORK2" library="TiLDA Mk3 Parts" package="TILDA_MKπ_ARTWORK_FRONT" value="ARTWORK_MKπ_FRONT" x="0" y="0"/>
 </elements>
 <signals>
