File: Mk3 v3.1415926535.sch (EAGLE design)
At the start: 150 parts, among them IC1 TPD3E001DRL, IC2 TPS62082, IC3 STM32F401V, IC4 BQ24092, IC6 CC3100MOD, IC7 BQ2970, IC8 LSM6DS3, IC9 LIS3MDL, J1 ZX62-AB-5PA(11), J2 ER-CON50HT-1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

Commit message: Library updates
Parts:
- LOGO3: value MICROPYTHON-STOP -> MICROPYTHON-SILK; device TiLDA Mk3 Parts:MICROPYTHON-STOP -> TiLDA Mk3 Parts:MICROPYTHON-SILK
Changed lines of the file:
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@@
 <variant name="L4" populate="no"/>
 </part>
-<part name="LOGO3" library="TiLDA Mk3 Parts" deviceset="MICROPYTHON" device="-STOP">
+<part name="LOGO3" library="TiLDA Mk3 Parts" deviceset="MICROPYTHON" device="-SILK" value="MICROPYTHON-SILK">
 <variant name="L4" populate="no"/>
 </part>
