File: Mk3 v3.1415926535.sch (EAGLE design)
At the start: 154 parts, among them IC1 TPD3E001DRL, IC2 TPS62082, IC3 STM32L475VG, IC4 BQ24092, IC6 CC3100MOD-LWK, IC7 BQ2970, IC8 LSM6DS3, IC9 LIS3MDL, J1 ZX62-AB-5PA(11), J2 ER-CON50HT-1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

Commit message: Update all values for L4 variant by default
Parts:
- ANT1: value CHIPANT -> 2450AT42A100E
- C19: value 0603/100n/10V/X5R or 0 ohm -> 0603/0R
- C29: value 0603/2.2u/6.3V/X5R -> 0603/100n/10V/X5R
- C48: value 0603/100n/10V/X5R -> DNP (0603/100n/10V/X5R)
- C9: value 0603/2.2u/6.3V/X5R or DNP -> DNP
- IC6: value CC3100MOD-LWK -> CC3100MOD
- IC7: value BQ2970 -> DNP (BQ2970)
- J3: value 2x5 1.27mm -> 2x5 1.27mm (NP)
- JP1, JP2: value M11PTH -> (NP)
- JP4: value TC2030-SWDNL -> (NP)
- L2, L3: value Bead -> BLM18KG121TN1D
- LOGO1: value OSHW-LOGOM -> OSHW-LOGOM (NP)
- LOGO2: value LOGO_TI-4MM -> LOGO_TI-4MM (NP)
- LOGO3: value LOGO_ST-4MM -> LOGO_ST-4MM (NP)
- LOGO4: value LOGO_HCD-4MM -> LOGO_HCD-4MM (NP)
- LOGO5: value LOGO_MICROSOFT-4MM -> LOGO_MICROSOFT-4MM (NP)
- LOGO6: value LOGO_MICROPYTHON-8MM -> LOGO_MICROPYTHON-8MM (NP)
- OUTLINE1: value TILDA_MK3_BOARDOUTLINE -> TILDA_MK3 (NP)
- Q4: value CSD85301Q2 -> DNP (CSD85301Q2)
- R12: value 0603/150/5% -> 0603/150R/5%
- R14, R26: value 0603/120/5% -> 0603/120R/5%
- R2: value 0603/330/5% -> 0603/1k/5%
- R28, R29: value 0603/4M7/5% -> DNP (0603/4M7/5%)
- R32: value DNP (0603/0R/5%) -> 0603/0R
- R50: value 0603/2k/5% -> DNP (0603/2k/5%)
- R51: value 0603/330/5% -> DNP (0603/330/5%)
- R7: value DNP or 0603/0R/5% -> 0603/0R
- R8: value DNP or 0 -> DNP
- S5: value Power Switch -> CUS-12TB
- S7: EBAY 272150658613 -> (none)
- SJ1: value SOLDERJUMPERNO -> OTG (NP)
- SV2, SV3, SV4, SV5, SV6, SV7: value (none) -> (NP)
- SW1: value JOYSTICK_MINI_MULTICOM_NOSILK -> JOYSTICK
- TP1, TP11, TP12, TP13, TP14, TP15, TP16, TP17, TP18, TP19, TP2, TP20, TP21, TP3, TP4, TP5: value TPB1,27 -> (NP)
- U1: value USD-SOCKET-SDIO -> USD-SOCKET
- U2: value ER-TFT024-3 -> ER-TFT024-3 (NP)
Connections:
- net CC_HIB renamed !CC_HIB
- net CC_RST renamed !CC_RST
- net N$17 renamed FORCE_AP
- net N$39 renamed !UART_CTS
- net N$41 renamed SOP2
- net N$43 renamed CC_RESERVED
- net N$44 renamed !UART_RTS
- net N$61 renamed TEST_58
- net N$65 renamed TEST_59
- net N$66 renamed TEST_60
- net N$67 renamed TEST_62
Other:
- moved on the sheet: LED1, Q3, R1, R20, R27, TP11

Commit message: Updating LED resistor values
Parts:
- R12: value 0603/150R/5% -> 0603/2k/5%
- R14: value 0603/120R/5% -> 0603/4k7/5%
- R2: value 0603/1k/5% -> 0603/4k7/5%
- R5: value 0603/2M2/5% -> 0603/4M7/5%
Changed lines of the file:
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@@
 <attribute name="FARNELL" value="2449874"/>
 </part>
-<part name="R2" library="TiLDA Mk3 Parts" deviceset="R-EU_" device="0603K-SMALL" value="0603/1k/5%"/>
+<part name="R2" library="TiLDA Mk3 Parts" deviceset="R-EU_" device="0603K-SMALL" value="0603/4k7/5%"/>
 <part name="S5" library="TiLDA Mk3 Parts" deviceset="SWITCH-SPST" device="-SMD-A" value="CUS-12TB">
 <attribute name="FARNELL" value="9575146"/>
@@
 </part>
 <part name="C13" library="TiLDA Mk3 Parts" deviceset="C-EU" device="C0603K-SMALL" value="0603/1u/10V/X5R"/>
-<part name="R5" library="TiLDA Mk3 Parts" deviceset="R-EU_" device="0603K-SMALL" value="0603/2M2/5%"/>
+<part name="R5" library="TiLDA Mk3 Parts" deviceset="R-EU_" device="0603K-SMALL" value="0603/4M7/5%"/>
 <part name="+3V10" library="TiLDA Mk3 Parts" deviceset="+3V3" device=""/>
 <part name="GND72" library="TiLDA Mk3 Parts" deviceset="GND" device=""/>
@@
 <attribute name="FARNELL" value="2426215"/>
 </part>
-<part name="R12" library="TiLDA Mk3 Parts" deviceset="R-EU_" device="0603K-SMALL" value="0603/150R/5%"/>
-<part name="R14" library="TiLDA Mk3 Parts" deviceset="R-EU_" device="0603K-SMALL" value="0603/120R/5%"/>
+<part name="R12" library="TiLDA Mk3 Parts" deviceset="R-EU_" device="0603K-SMALL" value="0603/2k/5%"/>
+<part name="R14" library="TiLDA Mk3 Parts" deviceset="R-EU_" device="0603K-SMALL" value="0603/4k7/5%"/>
 <part name="GND100" library="TiLDA Mk3 Parts" deviceset="GND" device=""/>
 <part name="GND101" library="TiLDA Mk3 Parts" deviceset="GND" device=""/>

Commit message: Correct joystick trace names
Parts:
- R18, R19: value DNP (0603/10k/5%) -> 0603/4k7/5%
Connections:
- net JOY_DOWN: now also IC3_PD.PD9, SW1.DOWN; no longer IC3_PD.PD10, SW1.LEFT
- net JOY_LEFT: now also IC3_PD.PD6, SW1.RIGHT; no longer IC3_PD.PD9, SW1.DOWN
- net JOY_RIGHT: now also IC3_PD.PD10, SW1.LEFT; no longer IC3_PD.PD6, SW1.RIGHT
Changed lines of the file:
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@@
 <part name="+3V1" library="TiLDA Mk3 Parts" deviceset="+3V3" device=""/>
 <part name="+3V2" library="TiLDA Mk3 Parts" deviceset="+3V3" device=""/>
-<part name="R18" library="TiLDA Mk3 Parts" deviceset="R-EU_" device="0603K-SMALL" value="DNP (0603/10k/5%)"/>
-<part name="R19" library="TiLDA Mk3 Parts" deviceset="R-EU_" device="0603K-SMALL" value="DNP (0603/10k/5%)"/>
+<part name="R18" library="TiLDA Mk3 Parts" deviceset="R-EU_" device="0603K-SMALL" value="0603/4k7/5%"/>
+<part name="R19" library="TiLDA Mk3 Parts" deviceset="R-EU_" device="0603K-SMALL" value="0603/4k7/5%"/>
 <part name="+3V3" library="TiLDA Mk3 Parts" deviceset="+3V3" device=""/>
 <part name="R28" library="TiLDA Mk3 Parts" deviceset="R-EU_" device="0603K-SMALL" value="DNP (0603/4M7/5%)">
@@
 </segment>
 </net>
-<net name="JOY_RIGHT" class="0">
+<net name="JOY_LEFT" class="0">
 <segment>
 <pinref part="IC3" gate="_PD" pin="PD6"/>
@@
 </segment>
 </net>
-<net name="JOY_LEFT" class="0">
+<net name="JOY_DOWN" class="0">
 <segment>
 <pinref part="IC3" gate="_PD" pin="PD9"/>
@@
 </segment>
 </net>
-<net name="JOY_DOWN" class="0">
+<net name="JOY_RIGHT" class="0">
 <segment>
 <pinref part="IC3" gate="_PD" pin="PD10"/>
